File: PCB_CAT_Vending_Machine_V1.0.kicad_pcb (KiCad board)
At the start: 2 copper layers, 108 x 129 mm, 279 parts, among them J1 12Vin, J10 Load, J11 Load, J12 Load, J13 Load, J14 Load, J15 Load, J16 Load, J17 Load, J18 Connector 4P, J19 Connector 4P, J2 Connector 4P, J20 Connector 4P, J21 Connector 3P, J22 Connector 3P, J23 Connector 4P, J24 Connector 4P, J25 Connector 4P, J26 Connector 4P, J27 Connector 4P, J28 Connector 4P, J29 Connector 4P, J3 Connector 4P, J30 Connector2P, J4 Connector 4P, J5 Connector 4P, J6 Connector 4P, J7 Connector 4P, J8 Connector 4P, J9 Connector 4P, Q1 2N7002, Q10 PT15-21C/TR8, Q12 AO3400A, Q13 AO3400A, Q14 AO3400A, Q15 AO3400A, Q16 AO3400A, Q17 AO3400A, Q18 AO3400A, Q2 2N7002, Q3 AO3400A, Q4 2N7002, Q5 2N7002, Q6 2N7002, Q7 2N7002, Q8 2N7002, Q9 2N7002, SW1 Pairing, SW2 Add 10 BTH, U1 ESP32-S3-N16R8-Module, U10 PC817C-S, U11 PC817C-S, U12 PC817C-S, U13 PCA9557PW, U14 PCA9557PW, U2 PCA9557PW, U3 PCA9557PW, U4 TPS5430DDA, U5 PC817C-S, U6 PC817C-S, U7 PC817C-S, U8 PC817C-S, U9 PC817C-S

Commit message: Frab1
Parts:
- removed JP1: Bankenote Selector, Jumper:SolderJumper-3_P1.3mm_Open_RoundedPad1.0x1.5mm
- added JP2: Jumper_Banknote, Connector_PinHeader_2.54mm:PinHeader_1x03_P2.54mm_Vertical, F.Cu at (65.0, 41.5)
- SW1: value Pairing -> Button
- SW2: value Add 10 BTH -> Button
- moved H4 17.5 mm to (119.5, 127.5)
- moved J2 7.50 mm to (24.5, 69.4), turned to 0 degrees
- moved J6 7.50 mm to (24.5, 105.8), turned to 0 degrees
- moved J7 7.50 mm to (24.5, 114.8), turned to 0 degrees
- moved J5 7.50 mm to (24.5, 96.7), turned to 0 degrees
- moved J8 7.50 mm to (24.5, 123.9), turned to 0 degrees
- moved J3 7.50 mm to (24.5, 78.5), turned to 0 degrees
- moved J4 7.50 mm to (24.5, 87.5), turned to 0 degrees
- moved J9 7.50 mm to (24.5, 133.0), turned to 0 degrees
- moved C49 4.30 mm to (116.0, 105.2)
- moved D16 4.30 mm to (113.5, 117.7)
- moved D8 4.30 mm to (122.3, 109.9)
- moved J16 4.30 mm to (120.1, 117.7)
- moved Q17 4.30 mm to (116.0, 108.8)
- moved R12 4.30 mm to (113.5, 115.2)
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Connections:
- J1 pad 1: GND -> +12V
- J1 pad 2: +12V -> GND
- J2 pad 1: /Connector/BTN0/12V_BTN0 -> +12V
- J2 pad 2: +12V -> /Connector/BTN0/GND_LED0
- J2 pad 3: /Connector/BTN0/GND_LED0 -> +12V
- J2 pad 4: +12V -> /Connector/BTN0/12V_BTN0
- J3 pad 1: /Connector/BTN1/12V_BTN1 -> +12V
- J3 pad 2: +12V -> /Connector/BTN1/GND_LED1
- J3 pad 3: /Connector/BTN1/GND_LED1 -> +12V
- J3 pad 4: +12V -> /Connector/BTN1/12V_BTN1
- J4 pad 1: /Connector/BTN2/12V_BTN2 -> +12V
- J4 pad 2: +12V -> /Connector/BTN2/GND_LED2
- J4 pad 3: /Connector/BTN2/GND_LED2 -> +12V
- J4 pad 4: +12V -> /Connector/BTN2/12V_BTN2
- J5 pad 1: /Connector/BTN3/12V_BTN3 -> +12V
- J5 pad 2: +12V -> /Connector/BTN3/GND_LED3
- J5 pad 3: /Connector/BTN3/GND_LED3 -> +12V
- J5 pad 4: +12V -> /Connector/BTN3/12V_BTN3
- J6 pad 1: /Connector/BTN4/12V_BTN4 -> +12V
- J6 pad 2: +12V -> /Connector/BTN4/GND_LED4
- J6 pad 3: /Connector/BTN4/GND_LED4 -> +12V
- J6 pad 4: +12V -> /Connector/BTN4/12V_BTN4
- J7 pad 1: /Connector/BTN5/12V_BTN5 -> +12V
- J7 pad 2: +12V -> /Connector/BTN5/GND_LED5
- J7 pad 3: /Connector/BTN5/GND_LED5 -> +12V
- J7 pad 4: +12V -> /Connector/BTN5/12V_BTN5
- J8 pad 1: /Connector/BTN6/12V_BTN6 -> +12V
- J8 pad 2: +12V -> /Connector/BTN6/GND_LED6
- J8 pad 3: /Connector/BTN6/GND_LED6 -> +12V
- J8 pad 4: +12V -> /Connector/BTN6/12V_BTN6
- J9 pad 1: /Connector/BTN7/12V_BTN7 -> +12V
- J9 pad 2: +12V -> /Connector/BTN7/GND_LED7
- J9 pad 3: /Connector/BTN7/GND_LED7 -> +12V
- J9 pad 4: +12V -> /Connector/BTN7/12V_BTN7
- Q10 pad 1: /Microcontroller/LightSen -> GND
- Q10 pad 2: GND -> /Microcontroller/LightSen
Routing:
- net +12V: track 816.7 -> 811.5 mm, vias 49 -> 54
- net /Connector/BTN0/12V_BTN0: track 37.0 -> 40.7 mm
- net /Connector/LED1: track 58.2 -> 56.2 mm
- net /Connector/LED0: track 51.9 -> 49.9 mm
- net /Microcontroller/Bank_RX: track 90.2 -> 92.0 mm
- net /Connector/LED2: track 64.1 -> 62.6 mm
- net /Connector/LED3: track 70.1 -> 68.8 mm
- net /Connector/LD6: track 42.8 -> 41.6 mm
- net /Connector/LED4: track 76.1 -> 74.9 mm
- net /Connector/BTN2/12V_BTN2: track 40.5 -> 41.6 mm
- net /Connector/BTN3/12V_BTN3: track 45.2 -> 46.2 mm
- net GND: track 318.4 -> 317.8 mm, vias 898 -> 995
- net /Microcontroller/Pulse/Bank_TX: track 12.8 -> 13.3 mm
Other:
- board size 108 x 129 mm -> 107 x 128 mm
