File: PCB_CAT_Vending_Machine_V1.0.kicad_pcb (KiCad board)
At the start: 2 copper layers, 107 x 128 mm, 279 parts, among them J1 12Vin, J10 Load, J11 Load, J12 Load, J13 Load, J14 Load, J15 Load, J16 Load, J17 Load, J18 Connector 4P, J19 Connector 4P, J2 Connector 4P, J20 Connector 4P, J21 Connector 3P, J22 Connector 3P, J23 Connector 4P, J24 Connector 4P, J25 Connector 4P, J26 Connector 4P, J27 Connector 4P, J28 Connector 4P, J29 Connector 4P, J3 Connector 4P, J30 Connector2P, J4 Connector 4P, J5 Connector 4P, J6 Connector 4P, J7 Connector 4P, J8 Connector 4P, J9 Connector 4P, Q1 2N7002, Q10 PT15-21C/TR8, Q12 AO3400A, Q13 AO3400A, Q14 AO3400A, Q15 AO3400A, Q16 AO3400A, Q17 AO3400A, Q18 AO3400A, Q2 2N7002, Q3 AO3400A, Q4 2N7002, Q5 2N7002, Q6 2N7002, Q7 2N7002, Q8 2N7002, Q9 2N7002, SW1 Button, SW2 Button, U1 ESP32-S3-N16R8-Module, U10 PC817C-S, U11 PC817C-S, U12 PC817C-S, U13 PCA9557PW, U14 PCA9557PW, U2 PCA9557PW, U3 PCA9557PW, U4 TPS5430DDA, U5 PC817C-S, U6 PC817C-S, U7 PC817C-S, U8 PC817C-S, U9 PC817C-S

Commit message: fix
Connections:
- R5 pad 2: +5V -> Net-(U4-VSENSE)
- SW1 pad 1: /Microcontroller/SW1 -> unconnected-(SW1-Pad1)
- SW1 pad 4: +3.3V -> unconnected-(SW1-A-Pad4)
- SW2 pad 1: /Microcontroller/SW2 -> unconnected-(SW2-Pad1)
- SW2 pad 4: +3.3V -> unconnected-(SW2-A-Pad4)
Routing:
- net +5V: track 226.4 -> 220.1 mm
- net +3.3V: track 638.5 -> 636.1 mm
- net Net-(U4-VSENSE): track 1.98 -> 4.28 mm
- net /Microcontroller/SW1: track 22.8 -> 20.6 mm
- net /Microcontroller/SW2: track 31.0 -> 28.8 mm
Changed lines of the file:
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@@
 	(net 173 "/Microcontroller/Bank_RX")
 	(net 174 "unconnected-(U1-GPIO11-Pad17)")
+	(net 175 "unconnected-(SW1-Pad1)")
+	(net 176 "unconnected-(SW1-A-Pad4)")
+	(net 177 "unconnected-(SW2-A-Pad4)")
+	(net 178 "unconnected-(SW2-Pad1)")
 	(footprint "Resistor_SMD:R_0402_1005Metric"
 		(layer "F.Cu")
@@
 			)
 		)
-		(property "Description" "Jumper, 3-pole, both open"
+		(property "Description" "-40℃~+105℃ 1 1kV 1x3P 2.54mm 2.5mm 3A 3P 3mm 6mm Brass Gold Pin Header Through Hole 插件,P=2.54mm Pin Headers ROHS"
 			(at 0 0 0)
 			(layer "F.Fab")
@@
 			)
 		)
+		(property "LCSC" "C52016391"
+			(at 0 0 180)
+			(unlocked yes)
+			(layer "F.Fab")
+			(hide yes)
+			(effects
+				(font
+					(size 1 1)
+					(thickness 0.15)
+				)
+			)
+		)
 		(property ki_fp_filters "Jumper* TestPoint*3Pads* TestPoint*Bridge*")
 		(sheetname "/Peripheral/")
 		(sheetfile "Peripheral.kicad_sch")
-		(attr through_hole exclude_from_bom)
+		(attr through_hole)
 		(fp_line
 			(start 1.38 1.27)
@@
 			(layers "F.Cu" "F.Mask" "F.Paste")
 			(roundrect_rratio 0.25)
-			(net 12 "+5V")
+			(net 36 "Net-(U4-VSENSE)")
 			(pintype "passive")
 		)
@@
 			(size 1.55 1.3)
 			(layers "F.Cu" "F.Mask" "F.Paste")
-			(net 114 "/Microcontroller/SW2")
+			(net 178 "unconnected-(SW2-Pad1)")
 			(pinfunction "1")
-			(pintype "passive")
+			(pintype "passive+no_connect")
 			(solder_mask_margin 0.102)
 		)
@@
 			(size 1.55 1.3)
 			(layers "F.Cu" "F.Mask" "F.Paste")
-			(net 11 "+3.3V")
+			(net 177 "unconnected-(SW2-A-Pad4)")
 			(pinfunction "A")
-			(pintype "passive")
+			(pintype "passive+no_connect")
 			(solder_mask_margin 0.102)
 		)
@@
 			(size 1.55 1.3)
 			(layers "F.Cu" "F.Mask" "F.Paste")
-			(net 113 "/Microcontroller/SW1")
+			(net 175 "unconnected-(SW1-Pad1)")
 			(pinfunction "1")
-			(pintype "passive")
+			(pintype "passive+no_connect")
 			(solder_mask_margin 0.102)
 		)
@@
 			(size 1.55 1.3)
 			(layers "F.Cu" "F.Mask" "F.Paste")
-			(net 11 "+3.3V")
+			(net 176 "unconnected-(SW1-A-Pad4)")
 			(pinfunction "A")
-			(pintype "passive")
+			(pintype "passive+no_connect")
 			(solder_mask_margin 0.102)
 		)
@@
 	)
 	(segment
-		(start 102.55 103.512501)
-		(end 98.05 103.512501)
-		(width 1)
-		(layer "F.Cu")
-		(net 11)
-	)
-	(segment
 		(start 83.375 100.775)
 		(end 82.1 102.05)
@@
 	)
 	(segment
+		(start 109.737499 103.5)
+		(end 109.75 103.512501)
+		(width 1)
+		(layer "F.Cu")
+		(net 11)
+	)
+	(segment
 		(start 77.309999 102.875)
 		(end 77.309999 103.472499)
@@
 	)
 	(segment
+		(start 101.4 103.5)
+		(end 102.537499 103.5)
+		(width 1)
+		(layer "F.Cu")
+		(net 11)
+	)
+	(segment
 		(start 68.9425 107.8)
 		(end 68.9425 107.0075)
@@
 	)
 	(segment
+		(start 108.6 103.5)
+		(end 109.737499 103.5)
+		(width 1)
+		(layer "F.Cu")
+		(net 11)
+	)
+	(segment
 		(start 97.75 39.609999)
 		(end 91.340001 39.609999)
@@
 	)
 	(segment
+		(start 102.537499 103.5)
+		(end 102.55 103.512501)
+		(width 1)
+		(layer "F.Cu")
+		(net 11)
+	)
+	(segment
 		(start 86.75 66.5)
 		(end 80.5 60.25)
@@
 	)
 	(segment
-		(start 102.55 103.512501)
-		(end 105.25 103.512501)
-		(width 1)
-		(layer "F.Cu")
-		(net 11)
-	)
-	(segment
 		(start 79.44 60.19)
 		(end 79.5 60.25)
@@
 	)
 	(segment
-		(start 109.75 103.512501)
-		(end 108.4 103.512501)
-		(width 1)
-		(layer "F.Cu")
-		(net 11)
-	)
-	(segment
 		(start 67.8 78.15)
 		(end 67.8 72.4)
@@
 	)
 	(segment
-		(start 108.4 103.512501)
-		(end 105.25 103.512501)
-		(width 1)
-		(layer "F.Cu")
-		(net 11)
-	)
-	(segment
 		(start 77.309999 103.472499)
 		(end 77.7375 103.9)
@@
 	)
 	(via
-		(at 100.25 103.55)
+		(at 101.4 103.5)
 		(size 0.6)
 		(drill 0.3)
@@
 	)
 	(via
-		(at 99.44 103.55)
+		(at 108.6 103.5)
 		(size 0.6)
 		(drill 0.3)
@@
 	)
 	(segment
-		(start 101.85 101.95)
-		(end 100.25 103.55)
-		(width 1)
-		(layer "B.Cu")
-		(net 11)
-	)
-	(segment
-		(start 99.44 103.55)
-		(end 100.25 103.55)
+		(start 95.1 92.8)
+		(end 95.1 60.25)
 		(width 1)
 		(layer "B.Cu")
@@
 	)
 	(segment
-		(start 95.1 92.8)
-		(end 95.1 60.25)
-		(width 1)
-		(layer "B.Cu")
-		(net 11)
-	)
-	(segment
 		(start 96.05 107.15)
 		(end 93.91 105.01)
@@
 	)
 	(segment
-		(start 101.85 99.55)
-		(end 101.85 101.95)
-		(width 1)
-		(layer "B.Cu")
-		(net 11)
-	)
-	(segment
-		(start 102.675 106.875)
-		(end 102.675 105.975)
-		(width 0.2)
-		(layer "B.Cu")
-		(net 11)
-	)
-	(segment
 		(start 58.8 31.05)
 		(end 58.8 36.85)
@@
 	)
 	(segment
+		(start 101.4 104.7)
+		(end 102.675 105.975)
+		(width 0.2)
+		(layer "B.Cu")
+		(net 11)
+	)
+	(segment
 		(start 95.1 46.4)
 		(end 82.2 33.5)
@@
 	)
 	(segment
-		(start 95.37 103.55)
-		(end 99.44 103.55)
+		(start 101.4 99.1)
+		(end 95.1 92.8)
 		(width 1)
 		(layer "B.Cu")
@@
 	)
 	(segment
-		(start 78.05 33.5)
-		(end 75.3 33.5)
+		(start 101.4 103.5)
+		(end 101.4 99.1)
 		(width 1)
 		(layer "B.Cu")
@@
 	)
 	(segment
-		(start 102.675 105.975)
-		(end 100.25 103.55)
-		(width 0.2)
+		(start 78.05 33.5)
+		(end 75.3 33.5)
+		(width 1)
 		(layer "B.Cu")
 		(net 11)
@@
 	)
 	(segment
-		(start 93.91 105.01)
-		(end 95.37 103.55)
+		(start 101.4 103.5)
+		(end 101.4 104.7)
+		(width 0.2)
+		(layer "B.Cu")
+		(net 11)
+	)
+	(segment
+		(start 101.4 103.5)
+		(end 95.42 103.5)
 		(width 1)
 		(layer "B.Cu")
@@
 	)
 	(segment
-		(start 101.85 99.55)
-		(end 95.1 92.8)
+		(start 102.675 105.975)
+		(end 102.675 106.875)
+		(width 0.2)
+		(layer "B.Cu")
+		(net 11)
+	)
+	(segment
+		(start 95.42 103.5)
+		(end 93.91 105.01)
 		(width 1)
 		(layer "B.Cu")
@@
 	)
 	(segment
+		(start 101.4 103.5)
+		(end 108.6 103.5)
+		(width 1)
+		(layer "B.Cu")
+		(net 11)
+	)
+	(segment
 		(start 77.3 102.05)
 		(end 77.3 104.35)
@@
 	)
 	(segment
-		(start 49.6 119.95)
-		(end 48.75 119.1)
-		(width 1)
-		(layer "F.Cu")
-		(net 12)
-	)
-	(segment
 		(start 51.4 103.4)
 		(end 65.1 103.4)
@@
 	)
 	(segment
-		(start 49.6 123.499999)
-		(end 49.6 119.95)
-		(width 1)
-		(layer "F.Cu")
-		(net 12)
-	)
-	(segment
 		(start 71.25 71.5)
 		(end 71.25 57.05)
@@
 	)
 	(segment
-		(start 49.6 123.499999)
-		(end 49.6 125.074999)
-		(width 1)
-		(layer "F.Cu")
-		(net 12)
-	)
-	(segment
 		(start 70.675 84.325)
 		(end 71.945 83.055)
@@
 	)
 	(segment
+		(start 49.6 123.499999)
+		(end 49.525002 123.499999)
+		(width 0.2)
+		(layer "F.Cu")
+		(net 36)
+	)
+	(segment
+		(start 49.525002 123.499999)
+		(end 47.95 125.075001)
+		(width 0.5)
+		(layer "F.Cu")
+		(net 36)
+	)
+	(segment
 		(start 48.144999 125.269999)
 		(end 47.95 125.075001)
@@
 	)
 	(segment
-		(start 102.265002 95.277502)
-		(end 102.550001 95.562501)
-		(width 0.2)
-		(layer "F.Cu")
-		(net 113)
-	)
-	(segment
-		(start 102.550001 95.562501)
-		(end 98.050001 95.562501)
-		(width 1)
-		(layer "F.Cu")
-		(net 113)
-	)
-	(segment
 		(start 102.265002 93.962501)
-		(end 102.265002 95.277502)
+		(end 98.255001 93.962501)
 		(width 0.2)
 		(layer "F.Cu")
@@
 	)
 	(segment
-		(start 109.49 93.962501)
-		(end 109.49 95.302502)
-		(width 0.2)
-		(layer "F.Cu")
-		(net 114)
-	)
-	(segment
-		(start 109.49 95.302502)
-		(end 109.749999 95.562501)
-		(width 0.2)
-		(layer "F.Cu")
-		(net 114)
-	)
-	(segment
 		(start 85.349998 96.325001)
 		(end 85.349998 97.592098)
@@
 	)
 	(segment
-		(start 90.875 96.725)
-		(end 104.087501 96.725)
+		(start 105.454999 93.962501)
+		(end 109.49 93.962501)
 		(width 0.2)
 		(layer "F.Cu")
@@
 	)
 	(segment
-		(start 109.749999 95.562501)
-		(end 105.249999 95.562501)
-		(width 1)
+		(start 90.875 96.725)
+		(end 104.087501 96.725)
+		(width 0.2)
 		(layer "F.Cu")
 		(net 114)
@@
 		(net 173)
 	)
+	(segment
+		(start 102.265002 95.277502)
+		(end 102.550001 95.562501)
+		(width 0.2)
+		(layer "F.Cu")
+		(net 175)
+	)
+	(segment
+		(start 109.49 95.302502)
+		(end 109.749999 95.562501)
+		(width 0.2)
+		(layer "F.Cu")
+		(net 178)
+	)
 	(zone

Commit message: to Kicad 10
Parts:
- added D34: SS84, Diode_SMD:D_SMC, F.Cu at (47.7, 145.2)
- moved C4 5.62 mm to (45.8, 138.0), turned to 180 degrees
- moved R5 3.31 mm to (46.4, 125.8), turned to 90 degrees
- moved C6 0.69 mm to (49.9, 135.0), turned to 135 degrees
Connections:
- J1 pad 1: +12V -> Net-(D34-A)
Routing:
- net GND: track 317.8 -> 272.7 mm, vias 995 -> 986
- net +12V: track 811.5 -> 777.3 mm, vias 54 -> 60
- net Net-(D34-A): track 0.00 -> 20.5 mm, vias 0 -> 4
- net Net-(U4-VSENSE): track 4.28 -> 3.57 mm
