File: BTNkicad_sch.kicad_sch (KiCad schematic)
At the start: 13 parts, among them Q1 2N7002, U12 PC817C-S

Commit message: SCH finish
Parts:
- R22, R80: value 4.7k -> 3k; LCSC C25900 -> C4211
Connections:
- net GND: now also Q1.2 (S); no longer Q1.3 (D)
- net GND_LED${No}: now also Q1.3 (D); no longer Q1.2 (S)
Other:
- moved on the sheet: Q1
Changed lines of the file:
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@@
-	(symbol
-		(lib_id "Device:R_Small")
-		(at 127 130.175 180)
-		(unit 1)
-		(exclude_from_sim no)
-		(in_bom yes)
-		(on_board yes)
-		(dnp no)
-		(property "Reference" "R22"
-			(at 129.54 130.175 0)
-			(effects
-				(font
-					(size 1.016 1.016)
-				)
-			)
-		)
-		(property "Value" "4.7k"
-			(at 127 130.175 90)
-			(effects
-				(font
-					(size 0.8 0.8)
-				)
-			)
-		)
-		(property "Footprint" "Resistor_SMD:R_0402_1005Metric"
-			(at 127 130.175 0)
-			(effects
-				(font
-					(size 1.27 1.27)
-				)
-				(hide yes)
-			)
-		)
-		(property "Datasheet" "-55℃~+155℃ 4.7kΩ 50V 62.5mW Thick Film Resistor ±1% ±100ppm/℃ 0402 Chip Resistor - Surface Mount ROHS"
-			(at 127 130.175 0)
-			(effects
-				(font
-					(size 1.27 1.27)
-				)
-				(hide yes)
-			)
-		)
-		(property "Description" "Resistor, small symbol"
-			(at 127 130.175 0)
-			(effects
-				(font
-					(size 1.27 1.27)
-				)
-				(hide yes)
-			)
-		)
-		(property "LCSC" "C25900"
-			(at 127 130.175 90)
-			(effects
-				(font
-					(size 1.27 1.27)
-				)
-				(hide yes)
-			)
-		)
-		(property "Link" ""
-			(at 127 130.175 0)
-			(effects
-				(font
-					(size 1.27 1.27)
-				)
-				(hide yes)
-			)
-		)
-		(pin "2"
-		)
-		(pin "1"
-		)
-		(instances
-			(project "PCB_CAT_Vending_Machine_V1.0"
-				(path "/f8bd6c94-f0e6-407f-98cc-e119e52a2f35/3b9c4b97-ebfa-4ac9-840a-ee2cf9f7cd88/0b2a77e9-14c2-4b88-bb12-8ec38d6907b4"
-					(reference "R68")
-					(unit 1)
-				)
-				(path "/f8bd6c94-f0e6-407f-98cc-e119e52a2f35/3b9c4b97-ebfa-4ac9-840a-ee2cf9f7cd88/1f662fc0-700e-4a53-8f25-29d5d6f99524"
-					(reference "R62")
-					(unit 1)
-				)
-				(path "/f8bd6c94-f0e6-407f-98cc-e119e52a2f35/3b9c4b97-ebfa-4ac9-840a-ee2cf9f7cd88/2eb76603-2d98-476b-9de6-9ee30cbab6b4"
-					(reference "R50")
-					(unit 1)
-				)
-				(path "/f8bd6c94-f0e6-407f-98cc-e119e52a2f35/3b9c4b97-ebfa-4ac9-840a-ee2cf9f7cd88/3b7d595c-aabc-4f1c-8bfc-e79b452a463e"
-					(reference "R44")
-					(unit 1)
-				)
-				(path "/f8bd6c94-f0e6-407f-98cc-e119e52a2f35/3b9c4b97-ebfa-4ac9-840a-ee2cf9f7cd88/45534c8c-de3d-430b-987d-7f352e5cf44d"
-					(reference "R56")
-					(unit 1)
-				)
-				(path "/f8bd6c94-f0e6-407f-98cc-e119e52a2f35/3b9c4b97-ebfa-4ac9-840a-ee2cf9f7cd88/5e38aab3-b28b-4dc5-a79b-6c7b0514426e"
-					(reference "R22")
-					(unit 1)
-				)
-				(path "/f8bd6c94-f0e6-407f-98cc-e119e52a2f35/3b9c4b97-ebfa-4ac9-840a-ee2cf9f7cd88/9cd2566d-f984-4948-abf0-8e9cce55fb0f"
-					(reference "R78")
-					(unit 1)
-				)
-				(path "/f8bd6c94-f0e6-407f-98cc-e119e52a2f35/3b9c4b97-ebfa-4ac9-840a-ee2cf9f7cd88/fdc5cd37-88e3-49d0-a95c-c565d851aa04"
-					(reference "R74")
-					(unit 1)
-				)
-			)
-		)
-	)
 	(symbol
 		(lib_id "Device:R_Small")
@@
 			)
 		)
-		(property "Value" "4.7k"
+		(property "Value" "3k"
 			(at 126.365 80.645 90)
 			(effects
@@
 			)
 		)
-		(property "Datasheet" "-55℃~+155℃ 4.7kΩ 50V 62.5mW Thick Film Resistor ±1% ±100ppm/℃ 0402 Chip Resistor - Surface Mount ROHS"
+		(property "Datasheet" "-55℃~+155℃ 100mW 3kΩ 75V Thick Film Resistor ±1% ±100ppm/℃ 0603 Chip Resistor - Surface Mount ROHS"
 			(at 126.365 80.645 0)
 			(effects
@@
 			)
 		)
-		(property "LCSC" "C25900"
+		(property "LCSC" "C4211 "
 			(at 126.365 80.645 90)
 			(effects
@@
 	(symbol
 		(lib_id "Transistor_FET:2N7002")
-		(at 137.16 84.455 270)
+		(at 137.16 84.455 90)
+		(mirror x)
 		(unit 1)
 		(exclude_from_sim no)
@@
 		(on_board yes)
 		(dnp no)
-		(fields_autoplaced yes)
 		(property "Reference" "Q1"
 			(at 137.16 90.805 90)
@@
 		)
 		(property "Footprint" "Package_TO_SOT_SMD:SOT-23"
-			(at 135.255 89.535 0)
+			(at 139.065 89.535 0)
 			(effects
 				(font
@@
 		)
 		(property "Datasheet" "https://www.onsemi.com/pub/Collateral/NDS7002A-D.PDF"
-			(at 133.35 89.535 0)
+			(at 140.97 89.535 0)
 			(effects
 				(font
@@
 					(unit 1)
 				)
+			)
+		)
+	)
+	(symbol
+		(lib_id "Device:R_Small")
+		(at 127 130.175 180)
+		(unit 1)
+		(exclude_from_sim no)
+		(in_bom yes)
+		(on_board yes)
+		(dnp no)
+		(property "Reference" "R22"
+			(at 129.54 130.175 0)
+			(effects
+				(font
+					(size 1.016 1.016)
+				)
+			)
+		)
+		(property "Value" "3k"
+			(at 127 130.175 90)
+			(effects
+				(font
+					(size 0.8 0.8)
+				)
+			)
+		)
+		(property "Footprint" "Resistor_SMD:R_0402_1005Metric"
+			(at 127 130.175 0)
+			(effects
+				(font
+					(size 1.27 1.27)
+				)
+				(hide yes)
+			)
+		)
+		(property "Datasheet" "-55℃~+155℃ 100mW 3kΩ 75V Thick Film Resistor ±1% ±100ppm/℃ 0603 Chip Resistor - Surface Mount ROHS"
+			(at 127 130.175 0)
+			(effects
+				(font
+					(size 1.27 1.27)
+				)
+				(hide yes)
+			)
+		)
+		(property "Description" "Resistor, small symbol"
+			(at 127 130.175 0)
+			(effects
+				(font
+					(size 1.27 1.27)
+				)
+				(hide yes)
+			)
+		)
+		(property "LCSC" "C4211 "
+			(at 127 130.175 90)
+			(effects
+				(font
+					(size 1.27 1.27)
+				)
+				(hide yes)
+			)
+		)
+		(property "Link" ""
+			(at 127 130.175 0)
+			(effects
+				(font
+					(size 1.27 1.27)
+				)
+				(hide yes)
+			)
+		)
+		(pin "2"
+		)
+		(pin "1"
+		)
+		(instances
+			(project "PCB_CAT_Vending_Machine_V1.0"
+				(path "/f8bd6c94-f0e6-407f-98cc-e119e52a2f35/3b9c4b97-ebfa-4ac9-840a-ee2cf9f7cd88/0b2a77e9-14c2-4b88-bb12-8ec38d6907b4"
+					(reference "R68")
+					(unit 1)
+				)
+				(path "/f8bd6c94-f0e6-407f-98cc-e119e52a2f35/3b9c4b97-ebfa-4ac9-840a-ee2cf9f7cd88/1f662fc0-700e-4a53-8f25-29d5d6f99524"
+					(reference "R62")
+					(unit 1)
+				)
+				(path "/f8bd6c94-f0e6-407f-98cc-e119e52a2f35/3b9c4b97-ebfa-4ac9-840a-ee2cf9f7cd88/2eb76603-2d98-476b-9de6-9ee30cbab6b4"
+					(reference "R50")
+					(unit 1)
+				)
+				(path "/f8bd6c94-f0e6-407f-98cc-e119e52a2f35/3b9c4b97-ebfa-4ac9-840a-ee2cf9f7cd88/3b7d595c-aabc-4f1c-8bfc-e79b452a463e"
+					(reference "R44")
+					(unit 1)
+				)
+				(path "/f8bd6c94-f0e6-407f-98cc-e119e52a2f35/3b9c4b97-ebfa-4ac9-840a-ee2cf9f7cd88/45534c8c-de3d-430b-987d-7f352e5cf44d"
+					(reference "R56")
+					(unit 1)
+				)
+				(path "/f8bd6c94-f0e6-407f-98cc-e119e52a2f35/3b9c4b97-ebfa-4ac9-840a-ee2cf9f7cd88/5e38aab3-b28b-4dc5-a79b-6c7b0514426e"
+					(reference "R22")
+					(unit 1)
+				)
+				(path "/f8bd6c94-f0e6-407f-98cc-e119e52a2f35/3b9c4b97-ebfa-4ac9-840a-ee2cf9f7cd88/9cd2566d-f984-4948-abf0-8e9cce55fb0f"
+					(reference "R78")
+					(unit 1)
+				)
+				(path "/f8bd6c94-f0e6-407f-98cc-e119e52a2f35/3b9c4b97-ebfa-4ac9-840a-ee2cf9f7cd88/fdc5cd37-88e3-49d0-a95c-c565d851aa04"
+					(reference "R74")
+					(unit 1)
+				)

Commit message: success
Parts:
- removed R80: 3k, Resistor_SMD:R_0402_1005Metric, symbol Device:R_Small
- added R29: 1k, Resistor_SMD:R_0402_1005Metric, symbol Device:R_Small
- C18: value 1nF -> 10nF; LCSC C1523 -> C15195
- C9: LCSC C15195 -> C15195
- R16: LCSC C25879 -> C25879
- R17: value 100k -> 10k; LCSC C25741 -> C25744
- R22: value 3k -> 1k; LCSC C4211 -> C11702
Connections:
- net +3.3V: now also R17.1
- net GND: no longer R17.2
- net GND_LED${No}: now also R29.1
- net LED${No}: now also R17.2; no longer R17.1
- net at D26.1 (K): now also R29.2

Commit message: to Kicad 10
Parts:
- R22, R29: LCSC C11702 -> C4109
