File: Connector.kicad_sch (KiCad schematic)
At the start: 16 parts, among them J10 Load_0, J11 Load_1, J12 Load_2, J13 Load_3, J14 Load_4, J15 Load_5, J16 Load_6, J17 Load_07, J2 Button_0, J3 Button_1, J4 Button_2, J5 Button_3, J6 Button_4, J7 Button_5, J8 Button_6, J9 Button_7

Commit message: success
Parts:
- J10: value Load_0 -> Load; Name (none) -> LD0
- J11: value Load_1 -> Load; Name (none) -> LD1
- J12: value Load_2 -> Load; Name (none) -> LD2
- J13: value Load_3 -> Load; Name (none) -> LD3
- J14: value Load_4 -> Load; Name (none) -> LD4
- J15: value Load_5 -> Load; Name (none) -> LD5
- J16: value Load_6 -> Load; Name (none) -> LD6
- J17: value Load_07 -> Load; Name (none) -> LD7
- J2: value Button_0 -> Connector 4P; LCSC C7429634 -> C7429634; Name (none) -> BTN0
- J3: value Button_1 -> Connector 4P; LCSC C7429634 -> C7429634; Name (none) -> BTN1
- J4: value Button_2 -> Connector 4P; LCSC C7429634 -> C7429634; Name (none) -> BTN2
- J5: value Button_3 -> Connector 4P; LCSC C7429634 -> C7429634; Name (none) -> BTN3
- J6: value Button_4 -> Connector 4P; LCSC C7429634 -> C7429634; Name (none) -> BTN4
- J7: value Button_5 -> Connector 4P; LCSC C7429634 -> C7429634; Name (none) -> BTN5
- J8: value Button_6 -> Connector 4P; LCSC C7429634 -> C7429634; Name (none) -> BTN6
- J9: value Button_7 -> Connector 4P; LCSC C7429634 -> C7429634; Name (none) -> BTN7
Connections:
- net +12V: now also J2.2 (Pin_2), J2.4 (Pin_4), J3.2 (Pin_2), J3.4 (Pin_4), J4.2 (Pin_2), J4.4 (Pin_4), J5.2 (Pin_2), J5.4 (Pin_4), J6.2 (Pin_2), J6.4 (Pin_4), J7.2 (Pin_2), J7.4 (Pin_4), J8.2 (Pin_2), J8.4 (Pin_4), J9.2 (Pin_2), J9.4 (Pin_4); no longer J2.1 (Pin_1), J2.3 (Pin_3), J3.1 (Pin_1), J3.3 (Pin_3), J4.1 (Pin_1), J4.3 (Pin_3), J5.1 (Pin_1), J5.3 (Pin_3), J6.1 (Pin_1), J6.3 (Pin_3), J7.1 (Pin_1), J7.3 (Pin_3), J8.1 (Pin_1), J8.3 (Pin_3), J9.1 (Pin_1), J9.3 (Pin_3)
- net BTN0/12V_BTN${No}: now also J2.1 (Pin_1); no longer J2.4 (Pin_4)
- net BTN0/GND_LED${No}: now also J2.3 (Pin_3); no longer J2.2 (Pin_2)
- net BTN1/12V_BTN${No}: now also J3.1 (Pin_1); no longer J3.4 (Pin_4)
- net BTN1/GND_LED${No}: now also J3.3 (Pin_3); no longer J3.2 (Pin_2)
- net BTN2/12V_BTN${No}: now also J4.1 (Pin_1); no longer J4.4 (Pin_4)
- net BTN2/GND_LED${No}: now also J4.3 (Pin_3); no longer J4.2 (Pin_2)
- net BTN3/12V_BTN${No}: now also J5.1 (Pin_1); no longer J5.4 (Pin_4)
- net BTN3/GND_LED${No}: now also J5.3 (Pin_3); no longer J5.2 (Pin_2)
- net BTN4/12V_BTN${No}: now also J6.1 (Pin_1); no longer J6.4 (Pin_4)
- net BTN4/GND_LED${No}: now also J6.3 (Pin_3); no longer J6.2 (Pin_2)
- net BTN5/12V_BTN${No}: now also J7.1 (Pin_1); no longer J7.4 (Pin_4)
- net BTN5/GND_LED${No}: now also J7.3 (Pin_3); no longer J7.2 (Pin_2)
- net BTN6/12V_BTN${No}: now also J8.1 (Pin_1); no longer J8.4 (Pin_4)
- net BTN6/GND_LED${No}: now also J8.3 (Pin_3); no longer J8.2 (Pin_2)
- net BTN7/12V_BTN${No}: now also J9.1 (Pin_1); no longer J9.4 (Pin_4)
- net BTN7/GND_LED${No}: now also J9.3 (Pin_3); no longer J9.2 (Pin_2)
- net Load0/12V_Load${No}: now also J10.2 (Pin_2); no longer J10.1 (Pin_1)
- net Load0/GND_Load${No}: now also J10.1 (Pin_1); no longer J10.2 (Pin_2)
- net Load1/12V_Load${No}: now also J11.2 (Pin_2); no longer J11.1 (Pin_1)
- net Load1/GND_Load${No}: now also J11.1 (Pin_1); no longer J11.2 (Pin_2)
- net Load2/12V_Load${No}: now also J12.2 (Pin_2); no longer J12.1 (Pin_1)
- net Load2/GND_Load${No}: now also J12.1 (Pin_1); no longer J12.2 (Pin_2)
- net Load3/12V_Load${No}: now also J13.2 (Pin_2); no longer J13.1 (Pin_1)
- net Load3/GND_Load${No}: now also J13.1 (Pin_1); no longer J13.2 (Pin_2)
- net Load4/12V_Load${No}: now also J14.2 (Pin_2); no longer J14.1 (Pin_1)
- net Load4/GND_Load${No}: now also J14.1 (Pin_1); no longer J14.2 (Pin_2)
- net Load5/12V_Load${No}: now also J15.2 (Pin_2); no longer J15.1 (Pin_1)
- net Load5/GND_Load${No}: now also J15.1 (Pin_1); no longer J15.2 (Pin_2)
- net Load6/12V_Load${No}: now also J16.2 (Pin_2); no longer J16.1 (Pin_1)
- net Load6/GND_Load${No}: now also J16.1 (Pin_1); no longer J16.2 (Pin_2)
- net Load7/12V_Load${No}: now also J17.2 (Pin_2); no longer J17.1 (Pin_1)
- net Load7/GND_Load${No}: now also J17.1 (Pin_1); no longer J17.2 (Pin_2)
Other:
- moved on the sheet: J10

Commit message: Frab1
Connections:
- net +12V: now also J2.1 (Pin_1), J2.3 (Pin_3), J3.1 (Pin_1), J3.3 (Pin_3), J4.1 (Pin_1), J4.3 (Pin_3), J5.1 (Pin_1), J5.3 (Pin_3), J6.1 (Pin_1), J6.3 (Pin_3), J7.1 (Pin_1), J7.3 (Pin_3), J8.1 (Pin_1), J8.3 (Pin_3), J9.1 (Pin_1), J9.3 (Pin_3); no longer J2.2 (Pin_2), J2.4 (Pin_4), J3.2 (Pin_2), J3.4 (Pin_4), J4.2 (Pin_2), J4.4 (Pin_4), J5.2 (Pin_2), J5.4 (Pin_4), J6.2 (Pin_2), J6.4 (Pin_4), J7.2 (Pin_2), J7.4 (Pin_4), J8.2 (Pin_2), J8.4 (Pin_4), J9.2 (Pin_2), J9.4 (Pin_4)
- net BTN0/12V_BTN${No}: now also J2.4 (Pin_4); no longer J2.1 (Pin_1)
- net BTN0/GND_LED${No}: now also J2.2 (Pin_2); no longer J2.3 (Pin_3)
- net BTN1/12V_BTN${No}: now also J3.4 (Pin_4); no longer J3.1 (Pin_1)
- net BTN1/GND_LED${No}: now also J3.2 (Pin_2); no longer J3.3 (Pin_3)
- net BTN2/12V_BTN${No}: now also J4.4 (Pin_4); no longer J4.1 (Pin_1)
- net BTN2/GND_LED${No}: now also J4.2 (Pin_2); no longer J4.3 (Pin_3)
- net BTN3/12V_BTN${No}: now also J5.4 (Pin_4); no longer J5.1 (Pin_1)
- net BTN3/GND_LED${No}: now also J5.2 (Pin_2); no longer J5.3 (Pin_3)
- net BTN4/12V_BTN${No}: now also J6.4 (Pin_4); no longer J6.1 (Pin_1)
- net BTN4/GND_LED${No}: now also J6.2 (Pin_2); no longer J6.3 (Pin_3)
- net BTN5/12V_BTN${No}: now also J7.4 (Pin_4); no longer J7.1 (Pin_1)
- net BTN5/GND_LED${No}: now also J7.2 (Pin_2); no longer J7.3 (Pin_3)
- net BTN6/12V_BTN${No}: now also J8.4 (Pin_4); no longer J8.1 (Pin_1)
- net BTN6/GND_LED${No}: now also J8.2 (Pin_2); no longer J8.3 (Pin_3)
- net BTN7/12V_BTN${No}: now also J9.4 (Pin_4); no longer J9.1 (Pin_1)
- net BTN7/GND_LED${No}: now also J9.2 (Pin_2); no longer J9.3 (Pin_3)
Other:
- moved on the sheet: J2, J3, J4, J5, J6, J7, J8, J9
