File: Load.kicad_sch (KiCad schematic)
At the start: 6 parts, among them Q3 AO3400A

Commit message: SCH finish
Parts:
- added C43: 1nF, Capacitor_SMD:C_0402_1005Metric, symbol Device:C_Small
- R1: value 4.7k -> 3k; LCSC C25900 -> C4211
Connections:
- net GND: now also C43.2
- net Load${No}: now also C43.1
Changed lines of the file:
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@@
+	)
+	(junction
+		(at 172.085 103.505)
+		(diameter 0)
+		(color 0 0 0 0)
+	)
+	(junction
+		(at 172.085 94.615)
+		(diameter 0)
+		(color 0 0 0 0)
 	)
 	(junction
@@
 	(wire
 		(pts
+			(xy 172.085 103.505) (xy 176.53 103.505)
+		)
+		(stroke
+			(width 0)
+			(type default)
+		)
+	)
+	(wire
+		(pts
 			(xy 133.35 91.44) (xy 134.62 91.44)
 		)
@@
 	(wire
 		(pts
-			(xy 167.64 94.615) (xy 173.355 94.615)
+			(xy 167.64 94.615) (xy 172.085 94.615)
+		)
+		(stroke
+			(width 0)
+			(type default)
+		)
+	)
+	(wire
+		(pts
+			(xy 172.085 101.6) (xy 172.085 103.505)
 		)
 		(stroke
@@
 	(wire
 		(pts
+			(xy 172.085 94.615) (xy 172.085 96.52)
+		)
+		(stroke
+			(width 0)
+			(type default)
+		)
+	)
+	(wire
+		(pts
 			(xy 133.35 86.995) (xy 133.35 91.44)
 		)
@@
 		(pts
 			(xy 127.635 100.965) (xy 128.905 100.965)
+		)
+		(stroke
+			(width 0)
+			(type default)
+		)
+	)
+	(wire
+		(pts
+			(xy 172.085 94.615) (xy 177.8 94.615)
 		)
 		(stroke
@@
 	(hierarchical_label "Load${No}"
 		(shape input)
-		(at 173.355 94.615 0)
+		(at 177.8 94.615 0)
 		(effects
 			(font
@@
 			)
 			(justify left)
+		)
+	)
+	(symbol
+		(lib_id "Device:R_Small")
+		(at 144.78 95.885 180)
+		(unit 1)
+		(exclude_from_sim no)
+		(in_bom yes)
+		(on_board yes)
+		(dnp no)
+		(property "Reference" "R1"
+			(at 147.32 95.885 0)
+			(effects
+				(font
+					(size 1.016 1.016)
+				)
+			)
+		)
+		(property "Value" "3k"
+			(at 144.78 95.885 90)
+			(effects
+				(font
+					(size 0.8 0.8)
+				)
+			)
+		)
+		(property "Footprint" "Resistor_SMD:R_0402_1005Metric"
+			(at 144.78 95.885 0)
+			(effects
+				(font
+					(size 1.27 1.27)
+				)
+				(hide yes)
+			)
+		)
+		(property "Datasheet" "-55℃~+155℃ 100mW 3kΩ 75V Thick Film Resistor ±1% ±100ppm/℃ 0603 Chip Resistor - Surface Mount ROHS"
+			(at 144.78 95.885 0)
+			(effects
+				(font
+					(size 1.27 1.27)
+				)
+				(hide yes)
+			)
+		)
+		(property "Description" "Resistor, small symbol"
+			(at 144.78 95.885 0)
+			(effects
+				(font
+					(size 1.27 1.27)
+				)
+				(hide yes)
+			)
+		)
+		(property "LCSC" "C4211 "
+			(at 144.78 95.885 90)
+			(effects
+				(font
+					(size 1.27 1.27)
+				)
+				(hide yes)
+			)
+		)
+		(property "Link" ""
+			(at 144.78 95.885 0)
+			(effects
+				(font
+					(size 1.27 1.27)
+				)
+				(hide yes)
+			)
+		)
+		(pin "2"
+		)
+		(pin "1"
+		)
+		(instances
+			(project "PCB_CAT_Vending_Machine_V1.0"
+				(path "/f8bd6c94-f0e6-407f-98cc-e119e52a2f35/3b9c4b97-ebfa-4ac9-840a-ee2cf9f7cd88/0c271627-317b-4a93-9f71-5e5c91d736bd"
+					(reference "R10")
+					(unit 1)
+				)
+				(path "/f8bd6c94-f0e6-407f-98cc-e119e52a2f35/3b9c4b97-ebfa-4ac9-840a-ee2cf9f7cd88/14d5d93e-bce6-49dd-948b-b629e32abd4c"
+					(reference "R1")
+					(unit 1)
+				)
+				(path "/f8bd6c94-f0e6-407f-98cc-e119e52a2f35/3b9c4b97-ebfa-4ac9-840a-ee2cf9f7cd88/587bad33-1d24-4ccb-8351-ab633d5a1fc5"
+					(reference "R11")
+					(unit 1)
+				)
+				(path "/f8bd6c94-f0e6-407f-98cc-e119e52a2f35/3b9c4b97-ebfa-4ac9-840a-ee2cf9f7cd88/5973e0c5-4c64-4f7f-805d-5b64c844a54c"
+					(reference "R2")
+					(unit 1)
+				)
+				(path "/f8bd6c94-f0e6-407f-98cc-e119e52a2f35/3b9c4b97-ebfa-4ac9-840a-ee2cf9f7cd88/7ab95cae-ce4f-4ab0-81c7-6a4d892e8f1f"
+					(reference "R13")
+					(unit 1)
+				)
+				(path "/f8bd6c94-f0e6-407f-98cc-e119e52a2f35/3b9c4b97-ebfa-4ac9-840a-ee2cf9f7cd88/9c642db8-62d1-4249-801c-ce7625f01657"
+					(reference "R8")
+					(unit 1)
+				)
+				(path "/f8bd6c94-f0e6-407f-98cc-e119e52a2f35/3b9c4b97-ebfa-4ac9-840a-ee2cf9f7cd88/d4d6f4ec-3715-476d-bb49-3a41bea4ec75"
+					(reference "R12")
+					(unit 1)
+				)
+				(path "/f8bd6c94-f0e6-407f-98cc-e119e52a2f35/3b9c4b97-ebfa-4ac9-840a-ee2cf9f7cd88/f491e371-fbc9-4f92-88ec-6d4cbb1d3331"
+					(reference "R3")
+					(unit 1)
+				)
+			)
+		)
+	)
+	(symbol
+		(lib_id "Device:C_Small")
+		(at 172.085 99.06 0)
+		(unit 1)
+		(exclude_from_sim no)
+		(in_bom yes)
+		(on_board yes)
+		(dnp no)
+		(property "Reference" "C43"
+			(at 174.625 97.79 0)
+			(effects
+				(font
+					(size 1 1)
+				)
+				(justify left)
+			)
+		)
+		(property "Value" "1nF"
+			(at 174.625 99.695 0)
+			(effects
+				(font
+					(size 1 1)
+				)
+				(justify left)
+			)
+		)
+		(property "Footprint" "Capacitor_SMD:C_0402_1005Metric"
+			(at 172.085 99.06 0)
+			(effects
+				(font
+					(size 1.27 1.27)
+				)
+				(hide yes)
+			)
+		)
+		(property "Datasheet" "1nF 50V X7R ±10% 0402 Multilayer Ceramic Capacitors MLCC - SMD/SMT ROHS"
+			(at 172.085 99.06 0)
+			(effects
+				(font
+					(size 1.27 1.27)
+				)
+				(hide yes)
+			)
+		)
+		(property "Description" "Unpolarized capacitor, small symbol"
+			(at 172.085 99.06 0)
+			(effects
+				(font
+					(size 1.27 1.27)
+				)
+				(hide yes)
+			)
+		)
+		(property "LCSC" "C1523"
+			(at 172.085 99.06 0)
+			(effects
+				(font
+					(size 1.27 1.27)
+				)
+				(hide yes)
+			)
+		)
+		(property "Link" ""
+			(at 172.085 99.06 0)
+			(effects
+				(font
+					(size 1.27 1.27)
+				)
+				(hide yes)
+			)
+		)
+		(pin "1"
+		)
+		(pin "2"
+		)
+		(instances
+			(project "PCB_CAT_Vending_Machine_V1.0"
+				(path "/f8bd6c94-f0e6-407f-98cc-e119e52a2f35/3b9c4b97-ebfa-4ac9-840a-ee2cf9f7cd88/0c271627-317b-4a93-9f71-5e5c91d736bd"
+					(reference "C47")
+					(unit 1)
+				)
+				(path "/f8bd6c94-f0e6-407f-98cc-e119e52a2f35/3b9c4b97-ebfa-4ac9-840a-ee2cf9f7cd88/14d5d93e-bce6-49dd-948b-b629e32abd4c"
+					(reference "C43")
+					(unit 1)
+				)
+				(path "/f8bd6c94-f0e6-407f-98cc-e119e52a2f35/3b9c4b97-ebfa-4ac9-840a-ee2cf9f7cd88/587bad33-1d24-4ccb-8351-ab633d5a1fc5"
+					(reference "C48")
+					(unit 1)
+				)
+				(path "/f8bd6c94-f0e6-407f-98cc-e119e52a2f35/3b9c4b97-ebfa-4ac9-840a-ee2cf9f7cd88/5973e0c5-4c64-4f7f-805d-5b64c844a54c"
+					(reference "C44")
+					(unit 1)
+				)
+				(path "/f8bd6c94-f0e6-407f-98cc-e119e52a2f35/3b9c4b97-ebfa-4ac9-840a-ee2cf9f7cd88/7ab95cae-ce4f-4ab0-81c7-6a4d892e8f1f"
+					(reference "C50")
+					(unit 1)
+				)
+				(path "/f8bd6c94-f0e6-407f-98cc-e119e52a2f35/3b9c4b97-ebfa-4ac9-840a-ee2cf9f7cd88/9c642db8-62d1-4249-801c-ce7625f01657"
+					(reference "C46")
+					(unit 1)
+				)
+				(path "/f8bd6c94-f0e6-407f-98cc-e119e52a2f35/3b9c4b97-ebfa-4ac9-840a-ee2cf9f7cd88/d4d6f4ec-3715-476d-bb49-3a41bea4ec75"
+					(reference "C49")
+					(unit 1)
+				)
+				(path "/f8bd6c94-f0e6-407f-98cc-e119e52a2f35/3b9c4b97-ebfa-4ac9-840a-ee2cf9f7cd88/f491e371-fbc9-4f92-88ec-6d4cbb1d3331"
+					(reference "C45")
+					(unit 1)
+				)
+			)
 		)
 	)
@@
 	(symbol
 		(lib_id "power:GND")
-		(at 172.085 103.505 90)
+		(at 176.53 103.505 90)
 		(unit 1)
 		(exclude_from_sim no)
@@
 		(dnp no)
 		(property "Reference" "#PWR033"
-			(at 178.435 103.505 0)
+			(at 182.88 103.505 0)
 			(effects
 				(font
@@
 		)
 		(property "Value" "GND"
-			(at 177.165 103.505 90)
+			(at 181.61 103.505 90)
 			(effects
 				(font
@@
 		)
 		(property "Footprint" ""
-			(at 172.085 103.505 0)
+			(at 176.53 103.505 0)
 			(effects
 				(font
@@
 		)
 		(property "Datasheet" ""
-			(at 172.085 103.505 0)
+			(at 176.53 103.505 0)
 			(effects
 				(font
@@
 		)
 		(property "Description" "Power symbol creates a global label with name \"GND\" , ground"
-			(at 172.085 103.505 0)
+			(at 176.53 103.505 0)
 			(effects
 				(font
@@
 					(unit 1)
 				)
-			)
-		)
-	)
-	(symbol
-		(lib_id "Device:R_Small")
-		(at 144.78 95.885 180)
-		(unit 1)
-		(exclude_from_sim no)
-		(in_bom yes)
-		(on_board yes)
-		(dnp no)
-		(property "Reference" "R1"
-			(at 147.32 95.885 0)
-			(effects
-				(font
-					(size 1.016 1.016)
-				)
-			)
-		)
-		(property "Value" "4.7k"
-			(at 144.78 95.885 90)
-			(effects
-				(font
-					(size 0.8 0.8)
-				)
-			)
-		)
-		(property "Footprint" "Resistor_SMD:R_0402_1005Metric"
-			(at 144.78 95.885 0)
-			(effects
-				(font
-					(size 1.27 1.27)
-				)
-				(hide yes)
-			)
-		)
-		(property "Datasheet" "-55℃~+155℃ 4.7kΩ 50V 62.5mW Thick Film Resistor ±1% ±100ppm/℃ 0402 Chip Resistor - Surface Mount ROHS"
-			(at 144.78 95.885 0)
-			(effects
-				(font
-					(size 1.27 1.27)
-				)
-				(hide yes)
-			)
-		)
-		(property "Description" "Resistor, small symbol"
-			(at 144.78 95.885 0)
-			(effects
-				(font
-					(size 1.27 1.27)
-				)
-				(hide yes)
-			)
-		)
-		(property "LCSC" "C25900"
-			(at 144.78 95.885 90)
-			(effects
-				(font
-					(size 1.27 1.27)
-				)
-				(hide yes)
-			)
-		)
-		(property "Link" ""
-			(at 144.78 95.885 0)
-			(effects
-				(font
-					(size 1.27 1.27)
-				)
-				(hide yes)
-			)
-		)
-		(pin "2"
-		)
-		(pin "1"
-		)
-		(instances
-			(project "PCB_CAT_Vending_Machine_V1.0"
-				(path "/f8bd6c94-f0e6-407f-98cc-e119e52a2f35/3b9c4b97-ebfa-4ac9-840a-ee2cf9f7cd88/0c271627-317b-4a93-9f71-5e5c91d736bd"
-					(reference "R10")
-					(unit 1)
-				)
-				(path "/f8bd6c94-f0e6-407f-98cc-e119e52a2f35/3b9c4b97-ebfa-4ac9-840a-ee2cf9f7cd88/14d5d93e-bce6-49dd-948b-b629e32abd4c"
-					(reference "R1")
-					(unit 1)
-				)
-				(path "/f8bd6c94-f0e6-407f-98cc-e119e52a2f35/3b9c4b97-ebfa-4ac9-840a-ee2cf9f7cd88/587bad33-1d24-4ccb-8351-ab633d5a1fc5"
-					(reference "R11")
-					(unit 1)
-				)
-				(path "/f8bd6c94-f0e6-407f-98cc-e119e52a2f35/3b9c4b97-ebfa-4ac9-840a-ee2cf9f7cd88/5973e0c5-4c64-4f7f-805d-5b64c844a54c"
-					(reference "R2")
-					(unit 1)
-				)
-				(path "/f8bd6c94-f0e6-407f-98cc-e119e52a2f35/3b9c4b97-ebfa-4ac9-840a-ee2cf9f7cd88/7ab95cae-ce4f-4ab0-81c7-6a4d892e8f1f"
-					(reference "R13")
-					(unit 1)
-				)
-				(path "/f8bd6c94-f0e6-407f-98cc-e119e52a2f35/3b9c4b97-ebfa-4ac9-840a-ee2cf9f7cd88/9c642db8-62d1-4249-801c-ce7625f01657"
-					(reference "R8")
-					(unit 1)
-				)
-				(path "/f8bd6c94-f0e6-407f-98cc-e119e52a2f35/3b9c4b97-ebfa-4ac9-840a-ee2cf9f7cd88/d4d6f4ec-3715-476d-bb49-3a41bea4ec75"
-					(reference "R12")
-					(unit 1)
-				)
-				(path "/f8bd6c94-f0e6-407f-98cc-e119e52a2f35/3b9c4b97-ebfa-4ac9-840a-ee2cf9f7cd88/f491e371-fbc9-4f92-88ec-6d4cbb1d3331"
-					(reference "R3")
-					(unit 1)
-				)

Commit message: success
Parts:
- removed R29: 100k, Resistor_SMD:R_0402_1005Metric, symbol Device:R_Small
- added R96: 10k, Resistor_SMD:R_0402_1005Metric, symbol Device:R_Small
- C43: value 1nF -> 10nF; LCSC C1523 -> C15195
- R1: value 3k -> 1k; LCSC C4211 -> C11702
Connections:
- net Load${No}: now also R96.2
- new net +3.3V: R96.1

Commit message: to Kicad 10
Parts:
- R1: LCSC C11702 -> C4109
