File: Microcontroller.kicad_sch (KiCad schematic)
At the start: 32 parts, among them SW1 Pairing, SW2 Add 10 BTH, U1 ESP32-S3-N16R8-Module, U13 PCA9557PW, U2 PCA9557PW, U3 PCA9557PW

Commit message: 3d
Changed lines of the file:
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@@
 	(bus
 		(pts
-			(xy 247.015 66.04) (xy 241.935 66.04)
-		)
-		(stroke
-			(width 0)
-			(type default)
-		)
-	)
-	(bus
-		(pts
 			(xy 102.235 99.695) (xy 102.235 102.235)
 		)
@@
 		)
 	)
+	(bus
+		(pts
+			(xy 254 67.945) (xy 248.92 67.945)
+		)
+		(stroke
+			(width 0)
+			(type default)
+		)
+	)
 	(wire
 		(pts
@@
 		)
 	)
-	(hierarchical_label "Water_Level{Trig Echo}"
+	(hierarchical_label "LD[0..7]"
 		(shape input)
-		(at 247.015 66.04 0)
+		(at 103.505 43.815 0)
 		(effects
 			(font
@@
 		)
 	)
-	(hierarchical_label "LD[0..7]"
+	(hierarchical_label "Water_Trigger[0..5]"
 		(shape input)
-		(at 103.505 43.815 0)
+		(at 254 67.945 0)
 		(effects
 			(font

Commit message: sch
Parts:
- added C41, C42: 100nF, Capacitor_SMD:C_0402_1005Metric, symbol Device:C_Small
- added R90: 10k, Resistor_SMD:R_0402_1005Metric, symbol Device:R_Small
- added U14: PCA9557PW, Package_SO:TSSOP-16_4.4x5mm_P0.65mm, symbol Interface_Expansion:PCA9557PW
Connections:
- net +3.3V: now also U3.4 (A1), C42.2, R90.1, U14.16 (VDD), U14.3 (A0), U14.4 (A1), U14.5 (A2)
- net GND: now also C41.2, C42.1, U14.8 (VSS); no longer U3.4 (A1)
- net I2C_SCL: now also U14.1 (SCL)
- net I2C_SDA: now also U14.2 (SDA)
- net SW1: now also U14.13 (IO6); no longer U1.41 (GPIO1)
- net SW2: now also U14.14 (IO7); no longer U1.40 (GPIO2)
- new net: C41.1, R90.2, U14.15 (~{RESET})
- new net Water_Trigger0: U14.6 (IO0)
- new net Water_Trigger1: U14.7 (IO1)
- new net Water_Trigger2: U14.9 (IO2)
- new net Water_Trigger3: U14.10 (IO3)
- new net Water_Trigger4: U14.11 (IO4)
- new net Water_Trigger5: U14.12 (IO5)
Other:
- moved on the sheet: C1, C10, C11, C12, C13, C14, C15, C16, C17, C2, C3, C33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

Commit message: SCH finish
Parts:
- added Q10: PT15-21C/TR8, LED_SMD:LED_1206_3216Metric, symbol Sensor_Optical:BPW42
- added R91: 10k, Resistor_SMD:R_0402_1005Metric, symbol Device:R_Small
Connections:
- net +3.3V: now also R91.2
- net GND: now also Q10.2 (E)
- net QR_Button0: now reaches U1.37 (GPIO40)
- net QR_Button1: now reaches U1.38 (GPIO41)
- net QR_Button2: now reaches U1.39 (GPIO42)
- net LightSen: now reaches U1.41 (GPIO1)
- net LightSen: now also Q10.1 (C), R91.1
Other:
- moved on the sheet: C1, C10, C11, C12, C13, C14, C15, C16, C17, C2, C3, C35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

Commit message: finish no review
Parts:
- added C51, C52, C53: 10nF, Capacitor_SMD:C_0402_1005Metric, symbol Device:C_Small
- added R92, R93, R94, R95: 10k, Resistor_SMD:R_0402_1005Metric, symbol Device:R_Small
Connections:
- net +3.3V: now also R95.1
- net BTN0: now also U3.9 (IO2); no longer U3.6 (IO0)
- net BTN1: now also U3.10 (IO3); no longer U3.7 (IO1)
- net BTN2: now also U3.11 (IO4); no longer U3.9 (IO2)
- net BTN3: now also U3.12 (IO5); no longer U3.10 (IO3)
- net BTN4: now also U3.13 (IO6); no longer U3.11 (IO4)
- net BTN5: now also U3.14 (IO7); no longer U3.12 (IO5)
- net BTN6: now also U3.7 (IO1); no longer U3.13 (IO6)
- net BTN7: now also U3.6 (IO0); no longer U3.14 (IO7)
- net COIN: now also U1.18 (GPIO12); no longer U1.17 (GPIO11)
- net GND: now also C51.1, C52.1, C53.1, R92.1, R93.1, R94.1
- net LD2: now also U2.10 (IO3); no longer U2.9 (IO2)
- net LD3: now also U2.9 (IO2); no longer U2.10 (IO3)
- net LD4: now also U2.12 (IO5); no longer U2.11 (IO4)
- net LD5: now also U2.11 (IO4); no longer U2.12 (IO5)
- net LD6: now also U2.14 (IO7); no longer U2.13 (IO6)
- net LD7: now also U2.13 (IO6); no longer U2.14 (IO7)
- net LED0: now also U13.14 (IO7); no longer U13.6 (IO0)
- net LED1: now also U13.13 (IO6); no longer U13.7 (IO1)
- net LED2: now also U13.12 (IO5); no longer U13.9 (IO2)
- net LED3: now also U13.11 (IO4); no longer U13.10 (IO3)
- net LED4: now also U13.10 (IO3); no longer U13.11 (IO4)
- net LED5: now also U13.9 (IO2); no longer U13.12 (IO5)
- net LED6: now also U13.7 (IO1); no longer U13.13 (IO6)
- net LED7: now also U13.6 (IO0); no longer U13.14 (IO7)
- net Pulse: now also U1.17 (GPIO11); no longer U1.18 (GPIO12)
- net QR_Button0: now also C53.2, R94.2
- net QR_Button1: now also C52.2, R93.2
- net QR_Button2: now also C51.2, R92.2
- net Water_Trigger0: now also U14.12 (IO5); no longer U14.6 (IO0)
- net Water_Trigger1: now also U14.11 (IO4); no longer U14.7 (IO1)
- net Water_Trigger2: now also U14.10 (IO3); no longer U14.9 (IO2)
- net Water_Trigger3: now also U14.9 (IO2); no longer U14.10 (IO3)
- net Water_Trigger4: now also U14.6 (IO0); no longer U14.11 (IO4)
- net Water_Trigger5: now also U14.7 (IO1); no longer U14.12 (IO5)
- net Door: now reaches U1.36 (GPIO39)
- net Door: now also R95.2
Other:
- moved on the sheet: Q10, R91

Commit message: success
Parts:
- added C54, C57, C58, C59, C60, C61, C62: 10nF, Capacitor_SMD:C_0402_1005Metric, symbol Device:C_Small
- added C55: 100nF, Capacitor_SMD:C_0402_1005Metric, symbol Device:C_Small
- added R100, R101, R102, R103, R98, R99: 10k, Resistor_SMD:R_0402_1005Metric, symbol Device:R_Small
- added R104, R105, R106, R107, R108, R109: 27k, Resistor_SMD:R_0603_1608Metric, symbol Device:R_Small
- added R110, R111, R112, R113, R114, R97: 220, Resistor_SMD:R_0402_1005Metric, symbol Device:R_Small
- added R115, R116, R123: 4.7k, Resistor_SMD:R_0402_1005Metric, symbol Device:R_Small
- C10, C11, C12, C13, C14, C15, C16, C17, C35, C36: LCSC C15195 -> C15195
- C51, C52, C53: value 10nF -> 100nF; LCSC C15195 -> C1525
- SW1: value Pairing -> Button; LCSC C7470157 -> C5340127; Name (none) -> Pairing
- SW2: value Add 10 BTH -> Button; LCSC C7470157 -> C5340127; Name (none) -> Add 10 BTH
Connections:
- net +3.3V: now also R92.1, R93.1, R94.1, R115.1, R116.1, R123.1
- net COIN: now also R123.2
- net Door: now also C55.1
- net GND: now also C54.2, C55.2, R100.1, R101.1, R102.1, R103.1, R98.1, R99.1; no longer R92.1, R93.1, R94.1
- net LightSen: now also C54.1
- net Water_Trigger0: now also R109.1; no longer U14.12 (IO5)
- net Water_Trigger1: now also R108.1; no longer U14.11 (IO4)
- net Water_Trigger2: now also R107.1; no longer U14.10 (IO3)
- net Water_Trigger3: now also R106.1; no longer U14.9 (IO2)
- net Water_Trigger4: now also R104.1; no longer U14.6 (IO0)
- net Water_Trigger5: now also R105.1; no longer U14.7 (IO1)
- net Pulse/Bank_TX: now reaches U1.4 (GPIO4)
- net Pulse/Bank_TX: now also R115.2
- net Bank_RX: now reaches U1.5 (GPIO5)
- net Bank_RX: now also R116.2
- net Pulse: no longer names the net of U1.17 (GPIO11)
- new net: R113.2, U14.11 (IO4)
- new net: R112.2, U14.10 (IO3)
- new net: R114.2, U14.12 (IO5)
- new net: R97.2, U14.6 (IO0)
- new net: R110.2, U14.7 (IO1)
- new net: R111.2, U14.9 (IO2)
- new net Water_Divider 0: C62.1, R103.2, R109.2, R114.1
- new net Water_Divider 1: C61.1, R102.2, R108.2, R113.1
- new net Water_Divider 2: C60.1, R101.2, R107.2, R112.1
- new net Water_Divider 3: C59.1, R100.2, R106.2, R111.1
- new net Water_Divider 4: C57.1, R104.2, R97.1, R98.2
- new net Water_Divider 5: C58.1, R105.2, R110.1, R99.2
- no-connect marks 12 -> 21
Other:
- moved on the sheet: C1, C2, C3, C35, C36, R6, R7, R92, R93, R94, SW1, SW2

Commit message: Frab1
Connections:
- net GND: now also Q10.1 (E); no longer Q10.2 (E)
- net LightSen: now also Q10.2 (C); no longer Q10.1 (C)

Commit message: fix
Connections:
- net +3.3V: no longer SW1.4 (A), SW2.4 (A)
- net SW1: no longer SW1.1
- net SW2: no longer SW2.1
- no-connect marks 21 -> 25
Other:
- moved on the sheet: SW1, SW2
Changed lines of the file:
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@@
 	)
 	(junction
-		(at 269.24 125.095)
-		(diameter 0)
-		(color 0 0 0 0)
-	)
-	(junction
 		(at 210.185 135.89)
 		(diameter 0)
@@
 	)
 	(junction
-		(at 269.24 148.59)
-		(diameter 0)
-		(color 0 0 0 0)
-	)
-	(junction
 		(at 255.27 101.6)
 		(diameter 0)
@@
 	)
 	(junction
-		(at 256.54 125.095)
-		(diameter 0)
-		(color 0 0 0 0)
-	)
-	(junction
 		(at 80.01 74.295)
 		(diameter 0)
@@
 	)
 	(junction
-		(at 256.54 148.59)
-		(diameter 0)
-		(color 0 0 0 0)
-	)
-	(junction
 		(at 255.27 106.68)
 		(diameter 0)
@@
 	)
 	(no_connect
+		(at 267.97 146.05)
+	)
+	(no_connect
 		(at 95.25 173.99)
 	)
 	(no_connect
+		(at 267.97 122.555)
+	)
+	(no_connect
+		(at 257.81 146.05)
+	)
+	(no_connect
 		(at 95.25 166.37)
 	)
@@
 		(at 95.25 161.29)
 	)
+	(no_connect
+		(at 257.81 122.555)
+	)
 	(bus_entry
 		(at 200.66 64.77)
@@
 	(wire
 		(pts
-			(xy 267.97 126.365) (xy 269.24 125.095)
-		)
-		(stroke
-			(width 0)
-			(type default)
-		)
-	)
-	(wire
-		(pts
 			(xy 151.765 105.41) (xy 151.765 107.95)
 		)
@@
 	(wire
 		(pts
-			(xy 254.635 148.59) (xy 256.54 148.59)
+			(xy 254.635 148.59) (xy 257.81 148.59)
 		)
 		(stroke
@@
 		)
 	)
-	(wire
-		(pts
-			(xy 256.54 125.095) (xy 257.81 126.365)
-		)
-		(stroke
-			(width 0)
-			(type default)
-		)
-	)
 	(bus
 		(pts
@@
 	(wire
 		(pts
-			(xy 269.24 125.095) (xy 271.145 125.095)
+			(xy 267.97 125.095) (xy 271.145 125.095)
 		)
 		(stroke
@@
 		)
 	)
-	(wire
-		(pts
-			(xy 269.24 148.59) (xy 267.97 147.32)
-		)
-		(stroke
-			(width 0)
-			(type default)
-		)
-	)
 	(bus
 		(pts
@@
 	(wire
 		(pts
-			(xy 254.635 125.095) (xy 256.54 125.095)
+			(xy 254.635 125.095) (xy 257.81 125.095)
 		)
 		(stroke
@@
 	(wire
 		(pts
-			(xy 256.54 148.59) (xy 257.81 149.86)
-		)
-		(stroke
-			(width 0)
-			(type default)
-		)
-	)
-	(wire
-		(pts
 			(xy 47.625 148.59) (xy 64.77 148.59)
 		)
@@
 	(wire
 		(pts
-			(xy 256.54 125.095) (xy 257.81 123.825)
-		)
-		(stroke
-			(width 0)
-			(type default)
-		)
-	)
-	(wire
-		(pts
 			(xy 186.055 41.91) (xy 182.88 41.91)
 		)
@@
 	(wire
 		(pts
-			(xy 269.24 148.59) (xy 271.145 148.59)
+			(xy 267.97 148.59) (xy 271.145 148.59)
 		)
 		(stroke
@@
 	(wire
 		(pts
-			(xy 267.97 149.86) (xy 269.24 148.59)
-		)
-		(stroke
-			(width 0)
-			(type default)
-		)
-	)
-	(wire
-		(pts
 			(xy 249.555 71.12) (xy 250.825 71.12)
 		)
@@
 	(wire
 		(pts
-			(xy 256.54 148.59) (xy 257.81 147.32)
-		)
-		(stroke
-			(width 0)
-			(type default)
-		)
-	)
-	(wire
-		(pts
 			(xy 90.17 87.63) (xy 99.695 87.63)
 		)
@@
 	(wire
 		(pts
-			(xy 271.145 121.285) (xy 271.145 125.095)
-		)
-		(stroke
-			(width 0)
-			(type default)
-		)
-	)
-	(wire
-		(pts
 			(xy 151.765 74.93) (xy 151.765 77.47)
 		)
@@
 	(wire
 		(pts
-			(xy 269.24 125.095) (xy 267.97 123.825)
+			(xy 271.145 125.095) (xy 271.145 121.285)
 		)
 		(stroke
@@
 	(symbol
 		(lib_id "Switch:SW_MEC_5E")
-		(at 262.89 149.86 0)
+		(at 262.89 148.59 0)
 		(unit 1)
 		(exclude_from_sim no)
@@
 		(dnp no)
 		(property "Reference" "SW2"
-			(at 262.89 140.97 0)
+			(at 262.89 139.7 0)
 			(effects
 				(font
@@
 		)
 		(property "Value" "Button"
-			(at 262.89 142.875 0)
+			(at 262.89 141.605 0)
 			(effects
 				(font
@@
 		)
 		(property "Footprint" "Sharing_IC_Footprint:430182043816"
-			(at 262.89 142.24 0)
+			(at 262.89 140.97 0)
 			(effects
 				(font
@@
 		)
 		(property "Datasheet" "http://www.apem.com/int/index.php?controller=attachment&id_attachment=1371"
-			(at 262.89 142.24 0)
+			(at 262.89 140.97 0)
 			(effects
 				(font
@@
 		)
 		(property "Description" "-25℃~+70℃ 100,000 cycles 12V 2.5N 50mA 6mm 6mm 8mm Black No Round Button SMD(SMT) Tab SPST Surface Mount,Vertical Without Bracket SMD-4P,6x6mm Tactile Switches ROHS"
-			(at 262.89 149.86 0)
+			(at 262.89 148.59 0)
 			(effects
 				(font
@@
 		)
 		(property "LCSC" " C5340127"
-			(at 262.89 149.86 0)
+			(at 262.89 148.59 0)
 			(effects
 				(font
@@
 		)
 		(property "Link" ""
-			(at 262.89 149.86 0)
+			(at 262.89 148.59 0)
 			(effects
 				(font
@@
 		)
 		(property "Name" "Add 10 BTH"
-			(at 262.89 149.86 0)
+			(at 262.89 148.59 0)
 			(effects
 				(font
@@
 	(symbol
 		(lib_id "Switch:SW_MEC_5E")
-		(at 262.89 126.365 0)
+		(at 262.89 125.095 0)
 		(unit 1)
 		(exclude_from_sim no)
@@
 		(dnp no)
 		(property "Reference" "SW1"
-			(at 262.89 117.475 0)
+			(at 262.89 116.205 0)
 			(effects
 				(font
@@
 		)
 		(property "Value" "Button"
-			(at 262.89 119.38 0)
+			(at 262.89 118.11 0)
 			(effects
 				(font
@@
 		)
 		(property "Footprint" "Sharing_IC_Footprint:430182043816"
-			(at 262.89 118.745 0)
+			(at 262.89 117.475 0)
 			(effects
 				(font
@@
 		)
 		(property "Datasheet" "http://www.apem.com/int/index.php?controller=attachment&id_attachment=1371"
-			(at 262.89 118.745 0)
+			(at 262.89 117.475 0)
 			(effects
 				(font
@@
 		)
 		(property "Description" "-25℃~+70℃ 100,000 cycles 12V 2.5N 50mA 6mm 6mm 8mm Black No Round Button SMD(SMT) Tab SPST Surface Mount,Vertical Without Bracket SMD-4P,6x6mm Tactile Switches ROHS"
-			(at 262.89 126.365 0)
+			(at 262.89 125.095 0)
 			(effects
 				(font
@@
 		)
 		(property "LCSC" " C5340127"
-			(at 262.89 126.365 0)
+			(at 262.89 125.095 0)
 			(effects
 				(font
@@
 		)
 		(property "Link" ""
-			(at 262.89 126.365 0)
+			(at 262.89 125.095 0)
 			(effects
 				(font
@@
 		)
 		(property "Name" "Pairing"
-			(at 262.89 126.365 0)
+			(at 262.89 125.095 0)
 			(effects
 				(font
