File: Peripheral.kicad_sch (KiCad schematic)
At the start: 6 parts, among them J18 Screen, J19 Banknote, J20 QR ESP32, J21 Coin, J22 RASPI, J23 Water Level

Commit message: 3d
Parts:
- added J24, J25, J26, J27, J28: Water Level, Connector_JST:JST_XH_B4B-XH-A_1x04_P2.50mm_Vertical, symbol Connector_Generic:Conn_01x04
Connections:
- net Water_Level.Trig is gone; now on net GND: J23.2 (Pin_2)
- net +12V: now also J23.4 (Pin_4), J24.4 (Pin_4), J25.4 (Pin_4), J26.4 (Pin_4), J27.4 (Pin_4), J28.4 (Pin_4)
- net +5V: no longer J23.1 (Pin_1)
- net GND: now also J24.2 (Pin_2), J25.2 (Pin_2), J26.2 (Pin_2), J27.2 (Pin_2), J28.2 (Pin_2); no longer J23.4 (Pin_4)
- net Water_Level.Echo renamed Water_Trigger0
- new net Water_Trigger1: J24.3 (Pin_3)
- new net Water_Trigger2: J25.3 (Pin_3)
- new net Water_Trigger3: J26.3 (Pin_3)
- new net Water_Trigger4: J27.3 (Pin_3)
- new net Water_Trigger5: J28.3 (Pin_3)
- no-connect marks 0 -> 6

Commit message: SCH finish
Parts:
- added J29: QR_Button, Connector_JST:JST_XH_B5B-XH-A_1x05_P2.50mm_Vertical, symbol Connector_Generic:Conn_01x05
Connections:
- net +3.3V: now also J29.1 (Pin_1)
- net GND: now also J29.5 (Pin_5)
- new net QR_Button0: J29.2 (Pin_2)
- new net QR_Button1: J29.3 (Pin_3)
- new net QR_Button2: J29.4 (Pin_4)

Commit message: finish no review
Parts:
- removed J29: QR_Button, Connector_JST:JST_XH_B5B-XH-A_1x05_P2.50mm_Vertical, symbol Connector_Generic:Conn_01x05
- added J29: QR_Button, Connector_JST:JST_XH_B4B-XH-A_1x04_P2.50mm_Vertical, symbol Connector_Generic:Conn_01x04
- added J30: DoorSensor, Connector_JST:JST_XH_B2B-XH-A_1x02_P2.50mm_Vertical, symbol Connector_Generic:Conn_01x02
- added R96: 100, Resistor_SMD:R_0402_1005Metric, symbol Device:R_Small
Connections:
- net +12V: now also J19.4 (Pin_4), J21.3 (Pin_3); no longer J19.1 (Pin_1), J21.1 (Pin_1)
- net +3.3V: now also J18.4 (Pin_4), J29.1 (Pin_1); no longer J18.1 (Pin_1)
- net +5V: now also J20.4 (Pin_4); no longer J20.1 (Pin_1)
- net GND: now also J18.3 (Pin_3), J19.1 (Pin_1), J19.3 (Pin_3), J20.1 (Pin_1), J21.1 (Pin_1), J30.2 (Pin_2); no longer J18.2 (Pin_2), J19.2 (Pin_2), J19.4 (Pin_4), J20.4 (Pin_4), J21.3 (Pin_3)
- net Pulse: now also J19.2 (Pin_2); no longer J19.3 (Pin_3)
- net QR_Button0: now also J29.2 (Pin_2)
- net QR_Button1: now also J29.3 (Pin_3)
- net QR_Button2: now also J29.4 (Pin_4)
- net Screen.CLK: now also J18.1 (Pin_1); no longer J18.4 (Pin_4)
- net Screen.DIO: now also J18.2 (Pin_2); no longer J18.3 (Pin_3)
- new net: J30.1 (Pin_1), R96.1
- new net Door: R96.2
Other:
- moved on the sheet: J18, J19, J20, J21, J22, J23, J24, J25, J26, J27, J28

Commit message: success
Parts:
- removed R96: 100, Resistor_SMD:R_0402_1005Metric, symbol Device:R_Small
- added JP1: Bankenote Selector, Jumper:SolderJumper-3_P1.3mm_Open_RoundedPad1.0x1.5mm, symbol Jumper:SolderJumper_3_Open
- J18: value Screen -> Connector 4P; LCSC C7429634 -> C7429634; Name (none) -> Screen
- J19: value Banknote -> Connector 4P; LCSC C7429634 -> C7429634; Name (none) -> Banknote
- J20: value QR ESP32 -> Connector 4P; LCSC C7429634 -> C7429634; Name (none) -> QR ESP32
- J21: value Coin -> Connector 3P; Name (none) -> Coin
- J22: value RASPI -> Connector 3P; Name (none) -> RASPI
- J23: value Water Level -> Connector 4P; LCSC C7429634 -> C7429634; Name (none) -> Water Level 0
- J24: value Water Level -> Connector 4P; LCSC C7429634 -> C7429634; Name (none) -> Water Level 1
- J25: value Water Level -> Connector 4P; LCSC C7429634 -> C7429634; Name (none) -> Water Level 2
- J26: value Water Level -> Connector 4P; LCSC C7429634 -> C7429634; Name (none) -> Water Level 3
- J27: value Water Level -> Connector 4P; LCSC C7429634 -> C7429634; Name (none) -> Water Level 4
- J28: value Water Level -> Connector 4P; LCSC C7429634 -> C7429634; Name (none) -> Water Level 5
- J29: value QR_Button -> Connector 4P; LCSC C7429634 -> C7429634; Name (none) -> QR_Button
- J30: value DoorSensor -> Connector2P; Name (none) -> DoorSensor
Connections:
- net +12V: now also J23.1 (Pin_1), J24.1 (Pin_1), J25.1 (Pin_1), J26.1 (Pin_1), J27.1 (Pin_1), J28.1 (Pin_1); no longer J23.4 (Pin_4), J24.4 (Pin_4), J25.4 (Pin_4), J26.4 (Pin_4), J27.4 (Pin_4), J28.4 (Pin_4)
- net +5V: now also J18.4 (Pin_4)
- net Door: now also J30.1 (Pin_1)
- net GND: now also J23.3 (Pin_3), J24.3 (Pin_3), J25.3 (Pin_3), J26.3 (Pin_3), J27.3 (Pin_3), J28.3 (Pin_3), J29.1 (Pin_1), JP1.3 (B); no longer J19.3 (Pin_3), J23.2 (Pin_2), J24.2 (Pin_2), J25.2 (Pin_2), J26.2 (Pin_2), J27.2 (Pin_2), J28.2 (Pin_2)
- net Water_Trigger0: now also J23.2 (Pin_2); no longer J23.3 (Pin_3)
- net Water_Trigger1: now also J24.2 (Pin_2); no longer J24.3 (Pin_3)
- net Water_Trigger2: now also J25.2 (Pin_2); no longer J25.3 (Pin_3)
- net Water_Trigger3: now also J26.2 (Pin_2); no longer J26.3 (Pin_3)
- net Water_Trigger4: now also J27.2 (Pin_2); no longer J27.3 (Pin_3)
- net Water_Trigger5: now also J28.2 (Pin_2); no longer J28.3 (Pin_3)
- removed net +3.3V: J18.4 (Pin_4), J29.1 (Pin_1)
- net Pulse renamed Bank_RX
- new net: J19.3 (Pin_3), JP1.2 (C)
- new net Pulse/Bank_TX: JP1.1 (A)
Other:
- moved on the sheet: J20, J21, J22, J23, J30

Commit message: Frab1
Parts:
- removed JP1: Bankenote Selector, Jumper:SolderJumper-3_P1.3mm_Open_RoundedPad1.0x1.5mm, symbol Jumper:SolderJumper_3_Open
- added JP2: Jumper_Banknote, Connector_PinHeader_2.54mm:PinHeader_1x03_P2.54mm_Vertical, symbol Jumper:Jumper_3_Open
Connections:
- net GND: now also JP2.3 (B)
- net Pulse/Bank_TX: now also JP2.1 (A)
- net at J19.3 (Pin_3): now also JP2.2 (C)
Changed lines of the file:
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@@
 	(wire
 		(pts
-			(xy 114.3 64.135) (xy 114.3 65.405)
+			(xy 114.3 65.405) (xy 114.3 66.675)
 		)
 		(stroke
@@
 	(wire
 		(pts
-			(xy 114.3 50.8) (xy 114.3 53.975)
+			(xy 114.3 50.8) (xy 114.3 52.705)
 		)
 		(stroke
@@
 	(symbol
 		(lib_id "power:GND")
-		(at 114.3 65.405 0)
+		(at 114.3 66.675 0)
 		(mirror y)
 		(unit 1)
@@
 		(dnp no)
 		(property "Reference" "#PWR098"
-			(at 114.3 71.755 0)
+			(at 114.3 73.025 0)
 			(effects
 				(font
@@
 		)
 		(property "Value" "GND"
-			(at 114.3 69.215 0)
+			(at 114.3 70.485 0)
 			(effects
 				(font
@@
 		)
 		(property "Footprint" ""
-			(at 114.3 65.405 0)
+			(at 114.3 66.675 0)
 			(effects
 				(font
@@
 		)
 		(property "Datasheet" ""
-			(at 114.3 65.405 0)
+			(at 114.3 66.675 0)
 			(effects
 				(font
@@
 		)
 		(property "Description" "Power symbol creates a global label with name \"GND\" , ground"
-			(at 114.3 65.405 0)
+			(at 114.3 66.675 0)
 			(effects
 				(font
@@
 				(path "/f8bd6c94-f0e6-407f-98cc-e119e52a2f35/9f2adda4-bc0e-4374-9492-404bc1f22ca7"
 					(reference "#PWR0148")
+					(unit 1)
+				)
+			)
+		)
+	)
+	(symbol
+		(lib_id "Jumper:Jumper_3_Open")
+		(at 114.3 59.055 270)
+		(unit 1)
+		(exclude_from_sim no)
+		(in_bom yes)
+		(on_board yes)
+		(dnp no)
+		(fields_autoplaced yes)
+		(property "Reference" "JP2"
+			(at 116.84 57.7849 90)
+			(effects
+				(font
+					(size 1.27 1.27)
+				)
+				(justify left)
+			)
+		)
+		(property "Value" "Jumper_Banknote"
+			(at 116.84 60.3249 90)
+			(effects
+				(font
+					(size 1.27 1.27)
+				)
+				(justify left)
+			)
+		)
+		(property "Footprint" "Connector_PinHeader_2.54mm:PinHeader_1x03_P2.54mm_Vertical"
+			(at 114.3 59.055 0)
+			(effects
+				(font
+					(size 1.27 1.27)
+				)
+				(hide yes)
+			)
+		)
+		(property "Datasheet" "~"
+			(at 114.3 59.055 0)
+			(effects
+				(font
+					(size 1.27 1.27)
+				)
+				(hide yes)
+			)
+		)
+		(property "Description" "-40℃~+105℃ 1 1kV 1x3P 2.54mm 2.5mm 3A 3P 3mm 6mm Brass Gold Pin Header Through Hole 插件,P=2.54mm Pin Headers ROHS"
+			(at 114.3 59.055 0)
+			(effects
+				(font
+					(size 1.27 1.27)
+				)
+				(hide yes)
+			)
+		)
+		(property "LCSC" "C52016391"
+			(at 114.3 59.055 90)
+			(effects
+				(font
+					(size 1.27 1.27)
+				)
+				(hide yes)
+			)
+		)
+		(pin "1"
+		)
+		(pin "2"
+		)
+		(pin "3"
+		)
+		(instances
+			(project ""
+				(path "/f8bd6c94-f0e6-407f-98cc-e119e52a2f35/9f2adda4-bc0e-4374-9492-404bc1f22ca7"
+					(reference "JP2")
 					(unit 1)
 				)
@@
 					(unit 1)
 				)
-			)
-		)
-	)
-	(symbol
-		(lib_id "Jumper:SolderJumper_3_Open")
-		(at 114.3 59.055 270)
-		(unit 1)
-		(exclude_from_sim no)
-		(in_bom no)
-		(on_board yes)
-		(dnp no)
-		(fields_autoplaced yes)
-		(property "Reference" "JP1"
-			(at 116.84 57.7849 90)
-			(effects
-				(font
-					(size 1.27 1.27)
-				)
-				(justify left)
-			)
-		)
-		(property "Value" "Bankenote Selector"
-			(at 116.84 60.3249 90)
-			(effects
-				(font
-					(size 1.27 1.27)
-				)
-				(justify left)
-			)
-		)
-		(property "Footprint" "Jumper:SolderJumper-3_P1.3mm_Open_RoundedPad1.0x1.5mm"
-			(at 114.3 59.055 0)
-			(effects
-				(font
-					(size 1.27 1.27)
-				)
-				(hide yes)
-			)
-		)
-		(property "Datasheet" "~"
-			(at 114.3 59.055 0)
-			(effects
-				(font
-					(size 1.27 1.27)
-				)
-				(hide yes)
-			)
-		)
-		(property "Description" "Solder Jumper, 3-pole, open"
-			(at 114.3 59.055 0)
-			(effects
-				(font
-					(size 1.27 1.27)
-				)
-				(hide yes)
-			)
-		)
-		(pin "2"
-		)
-		(pin "1"
-		)
-		(pin "3"
-		)
-		(instances
-			(project ""
-				(path "/f8bd6c94-f0e6-407f-98cc-e119e52a2f35/9f2adda4-bc0e-4374-9492-404bc1f22ca7"
-					(reference "JP1")
-					(unit 1)
-				)
