File: Power_supply.kicad_sch (KiCad schematic)
At the start: 11 parts, among them J1 12Vin, U4 TPS5430DDA

Commit message: finish no review
Connections:
- net +12V: now also J1.2 (Pin_2); no longer J1.1 (Pin_1)
- net GND: now also J1.1 (Pin_1); no longer J1.2 (Pin_2)
Other:
- moved on the sheet: J1
Changed lines of the file:
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@@
 	(symbol
 		(lib_id "Connector:Screw_Terminal_01x02")
-		(at 93.345 68.58 0)
-		(mirror y)
+		(at 93.345 71.12 180)
 		(unit 1)
 		(exclude_from_sim no)
@@
 		(dnp no)
 		(property "Reference" "J1"
-			(at 90.17 68.5799 0)
+			(at 90.17 71.1201 0)
 			(effects
 				(font
@@
 		)
 		(property "Value" "12Vin"
-			(at 90.17 71.1199 0)
+			(at 90.17 68.5801 0)
 			(effects
 				(font
@@
 		)
 		(property "Footprint" "Sharing_Connector_Footprint:CONN-TH_2P-P5.00_XY2500V-D-5.00-2P"
-			(at 93.345 68.58 0)
+			(at 93.345 71.12 0)
 			(effects
 				(font
@@
 		)
 		(property "Datasheet" "https://jlcpcb.com/api/file/downloadByFileSystemAccessId/8588888835996454912"
-			(at 93.345 68.58 0)
+			(at 93.345 71.12 0)
 			(effects
 				(font
@@
 		)
 		(property "Description" "1 15A 1x2P 2 2P 300V 5mm Board Side/Socket - Closed Green Hinged (Snap On) Through Hole Plugin,P=5mm Pluggable System Terminal Block ROHS"
-			(at 93.345 68.58 0)
+			(at 93.345 71.12 0)
 			(effects
 				(font
@@
 		)
 		(property "LCSC" "C505779"
-			(at 93.345 68.58 0)
+			(at 93.345 71.12 0)
 			(effects
 				(font
@@
 		)
 		(property "Link" ""
-			(at 93.345 68.58 0)
+			(at 93.345 71.12 0)
 			(effects
 				(font
@@
 		)
 		(instances
-			(project ""
+			(project "PCB_CAT_Vending_Machine_V1.0"
 				(path "/f8bd6c94-f0e6-407f-98cc-e119e52a2f35/a76cc5d0-f19b-45e7-b348-68021cdb7480"
 					(reference "J1")

Commit message: success
Parts:
- C4, C5: LCSC C696188 -> C696188
Changed lines of the file:
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@@
+	(wire
+		(pts
+			(xy 190.5 69.85) (xy 190.5 73.66)
+		)
+		(stroke
+			(width 0)
+			(type default)
+		)
+	)
 	(wire
 		(pts
@@
 		(pts
 			(xy 184.785 73.66) (xy 190.5 73.66)
+		)
+		(stroke
+			(width 0)
+			(type default)
+		)
+	)
+	(wire
+		(pts
+			(xy 121.285 66.675) (xy 121.285 68.58)
 		)
 		(stroke
@@
 			)
 		)
-		(property "LCSC" " C696188"
+		(property "LCSC" "C696188"
 			(at 190.5 79.375 0)
 			(effects
@@
 			)
 		)
-		(property "LCSC" " C696188"
+		(property "LCSC" "C696188"
 			(at 106.045 73.66 0)
 			(effects
@@
 	)
 	(symbol
+		(lib_id "power:PWR_FLAG")
+		(at 190.5 69.85 0)
+		(unit 1)
+		(exclude_from_sim no)
+		(in_bom yes)
+		(on_board yes)
+		(dnp no)
+		(fields_autoplaced yes)
+		(property "Reference" "#FLG01"
+			(at 190.5 67.945 0)
+			(effects
+				(font
+					(size 1.27 1.27)
+				)
+				(hide yes)
+			)
+		)
+		(property "Value" "PWR_FLAG"
+			(at 190.5 65.405 0)
+			(effects
+				(font
+					(size 1.27 1.27)
+				)
+			)
+		)
+		(property "Footprint" ""
+			(at 190.5 69.85 0)
+			(effects
+				(font
+					(size 1.27 1.27)
+				)
+				(hide yes)
+			)
+		)
+		(property "Datasheet" "~"
+			(at 190.5 69.85 0)
+			(effects
+				(font
+					(size 1.27 1.27)
+				)
+				(hide yes)
+			)
+		)
+		(property "Description" "Special symbol for telling ERC where power comes from"
+			(at 190.5 69.85 0)
+			(effects
+				(font
+					(size 1.27 1.27)
+				)
+				(hide yes)
+			)
+		)
+		(pin "1"
+		)
+		(instances
+			(project "PCB_CAT_Vending_Machine_V1.0"
+				(path "/f8bd6c94-f0e6-407f-98cc-e119e52a2f35/a76cc5d0-f19b-45e7-b348-68021cdb7480"
+					(reference "#FLG01")
+					(unit 1)
+				)
+			)
+		)
+	)
+	(symbol
 		(lib_id "power:GND")
 		(at 121.285 77.47 0)
@@
 					(unit 1)
 				)
+			)
+		)
+	)
+	(symbol
+		(lib_id "power:PWR_FLAG")
+		(at 121.285 66.675 0)
+		(unit 1)
+		(exclude_from_sim no)
+		(in_bom yes)
+		(on_board yes)
+		(dnp no)
+		(property "Reference" "#FLG02"
+			(at 121.285 64.77 0)
+			(effects
+				(font
+					(size 1.27 1.27)
+				)
+				(hide yes)
+			)
+		)
+		(property "Value" "PWR_FLAG"
+			(at 121.285 62.865 0)
+			(effects
+				(font
+					(size 1.27 1.27)
+				)
+			)
+		)
+		(property "Footprint" ""
+			(at 121.285 66.675 0)
+			(effects
+				(font
+					(size 1.27 1.27)
+				)
+				(hide yes)
+			)
+		)
+		(property "Datasheet" "~"
+			(at 121.285 66.675 0)
+			(effects
+				(font
+					(size 1.27 1.27)
+				)
+				(hide yes)
+			)
+		)
+		(property "Description" "Special symbol for telling ERC where power comes from"
+			(at 121.285 66.675 0)
+			(effects
+				(font
+					(size 1.27 1.27)
+				)
+				(hide yes)
+			)
+		)
+		(pin "1"
+		)
+		(instances
+			(project "PCB_CAT_Vending_Machine_V1.0"
+				(path "/f8bd6c94-f0e6-407f-98cc-e119e52a2f35/a76cc5d0-f19b-45e7-b348-68021cdb7480"
+					(reference "#FLG02")
+					(unit 1)
+				)

Commit message: Frab1
Connections:
- net +12V: now also J1.1 (Pin_1); no longer J1.2 (Pin_2)
- net GND: now also J1.2 (Pin_2); no longer J1.1 (Pin_1)
Other:
- moved on the sheet: J1
Changed lines of the file:
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@@
 	(symbol
 		(lib_id "Connector:Screw_Terminal_01x02")
-		(at 93.345 71.12 180)
+		(at 93.345 68.58 0)
+		(mirror y)
 		(unit 1)
 		(exclude_from_sim no)
@@
 		(dnp no)
 		(property "Reference" "J1"
-			(at 90.17 71.1201 0)
+			(at 90.17 68.5799 0)
 			(effects
 				(font
@@
 		)
 		(property "Value" "12Vin"
-			(at 90.17 68.5801 0)
+			(at 90.17 71.1199 0)
 			(effects
 				(font
@@
 		)
 		(property "Footprint" "Sharing_Connector_Footprint:CONN-TH_2P-P5.00_XY2500V-D-5.00-2P"
-			(at 93.345 71.12 0)
+			(at 93.345 68.58 0)
 			(effects
 				(font
@@
 		)
 		(property "Datasheet" "https://jlcpcb.com/api/file/downloadByFileSystemAccessId/8588888835996454912"
-			(at 93.345 71.12 0)
+			(at 93.345 68.58 0)
 			(effects
 				(font
@@
 		)
 		(property "Description" "1 15A 1x2P 2 2P 300V 5mm Board Side/Socket - Closed Green Hinged (Snap On) Through Hole Plugin,P=5mm Pluggable System Terminal Block ROHS"
-			(at 93.345 71.12 0)
+			(at 93.345 68.58 0)
 			(effects
 				(font
@@
 		)
 		(property "LCSC" "C505779"
-			(at 93.345 71.12 0)
+			(at 93.345 68.58 0)
 			(effects
 				(font
@@
 		)
 		(property "Link" ""
-			(at 93.345 71.12 0)
+			(at 93.345 68.58 0)
 			(effects
 				(font

Commit message: fix
Connections:
- net +5V: no longer R5.2
- net at R4.1, U4.4 (VSENSE): now also R5.2
Other:
- moved on the sheet: R4, R5
Changed lines of the file:
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@@
 	(text "0603"
 		(exclude_from_sim no)
-		(at 163.83 85.725 0)
+		(at 155.575 84.455 0)
 		(effects
 			(font
@@
 	(text "0603"
 		(exclude_from_sim no)
-		(at 159.385 80.645 0)
+		(at 161.29 80.645 0)
 		(effects
 			(font
@@
 			)
 		)
-	)
-	(junction
-		(at 165.1 78.74)
-		(diameter 0)
-		(color 0 0 0 0)
 	)
 	(junction
@@
 	)
 	(junction
+		(at 156.845 78.74)
+		(diameter 0)
+		(color 0 0 0 0)
+	)
+	(junction
 		(at 106.045 68.58)
 		(diameter 0)
@@
 	(wire
 		(pts
+			(xy 156.845 78.74) (xy 158.75 78.74)
+		)
+		(stroke
+			(width 0)
+			(type default)
+		)
+	)
+	(wire
+		(pts
 			(xy 142.24 85.725) (xy 140.97 86.995)
 		)
@@
 	(wire
 		(pts
-			(xy 165.1 78.74) (xy 170.18 78.74)
-		)
-		(stroke
-			(width 0)
-			(type default)
-		)
-	)
-	(wire
-		(pts
 			(xy 190.5 81.915) (xy 190.5 83.82)
 		)
@@
 	(wire
 		(pts
+			(xy 154.94 78.74) (xy 156.845 78.74)
+		)
+		(stroke
+			(width 0)
+			(type default)
+		)
+	)
+	(wire
+		(pts
 			(xy 106.045 68.58) (xy 121.285 68.58)
 		)
@@
 	(wire
 		(pts
-			(xy 165.1 86.995) (xy 165.1 88.265)
+			(xy 156.845 85.725) (xy 156.845 86.995)
 		)
 		(stroke
@@
 	(wire
 		(pts
-			(xy 154.94 78.74) (xy 156.845 78.74)
-		)
-		(stroke
-			(width 0)
-			(type default)
-		)
-	)
-	(wire
-		(pts
 			(xy 206.375 81.915) (xy 206.375 83.82)
 		)
@@
 	(wire
 		(pts
-			(xy 165.1 78.74) (xy 165.1 81.915)
+			(xy 156.845 78.74) (xy 156.845 80.645)
 		)
 		(stroke
@@
 	(wire
 		(pts
+			(xy 172.085 78.74) (xy 163.83 78.74)
+		)
+		(stroke
+			(width 0)
+			(type default)
+		)
+	)
+	(wire
+		(pts
 			(xy 190.5 73.66) (xy 190.5 76.835)
 		)
@@
 			(width 0)
 			(type default)
-		)
-	)
-	(wire
-		(pts
-			(xy 161.925 78.74) (xy 165.1 78.74)
-		)
-		(stroke
-			(width 0)
-			(type default)
-		)
-	)
-	(label "Vout_5V"
-		(at 170.18 78.74 180)
-		(effects
-			(font
-				(size 1.27 1.27)
-			)
-			(justify right bottom)
 		)
 	)
@@
 		)
 	)
+	(label "Vout_5V"
+		(at 172.085 78.74 180)
+		(effects
+			(font
+				(size 1.27 1.27)
+			)
+			(justify right bottom)
+		)
+	)
 	(symbol
 		(lib_id "Device:R_Small")
-		(at 165.1 84.455 180)
+		(at 156.845 83.185 180)
 		(unit 1)
 		(exclude_from_sim no)
@@
 		(dnp no)
 		(property "Reference" "R5"
-			(at 163.83 83.82 0)
+			(at 155.575 82.55 0)
 			(effects
 				(font
@@
 		)
 		(property "Value" "4.7k"
-			(at 165.1 84.455 90)
+			(at 156.845 83.185 90)
 			(effects
 				(font
@@
 		)
 		(property "Footprint" "Resistor_SMD:R_0603_1608Metric"
-			(at 165.1 84.455 0)
+			(at 156.845 83.185 0)
 			(effects
 				(font
@@
 		)
 		(property "Datasheet" "https://jlcpcb.com/api/file/downloadByFileSystemAccessId/8579706381320323072"
-			(at 165.1 84.455 0)
+			(at 156.845 83.185 0)
 			(effects
 				(font
@@
 		)
 		(property "Description" "-55℃~+155℃ 100mW 4.7kΩ 75V Thick Film Resistor ±1% ±100ppm/℃ 0603 Chip Resistor - Surface Mount ROHS"
-			(at 165.1 84.455 0)
+			(at 156.845 83.185 0)
 			(effects
 				(font
@@
 		)
 		(property "LCSC" "C23162"
-			(at 165.1 84.455 0)
+			(at 156.845 83.185 0)
 			(effects
 				(font
@@
 		)
 		(property "Link" ""
-			(at 165.1 84.455 0)
+			(at 156.845 83.185 0)
 			(effects
 				(font
@@
 	(symbol
 		(lib_id "power:GND")
-		(at 165.1 88.265 0)
+		(at 156.845 86.995 0)
 		(unit 1)
 		(exclude_from_sim no)
@@
 		(fields_autoplaced yes)
 		(property "Reference" "#PWR025"
-			(at 165.1 94.615 0)
+			(at 156.845 93.345 0)
 			(effects
 				(font
@@
 		)
 		(property "Value" "GND"
-			(at 165.1 92.71 0)
+			(at 156.845 91.44 0)
 			(effects
 				(font
@@
 		)
 		(property "Footprint" ""
-			(at 165.1 88.265 0)
+			(at 156.845 86.995 0)
 			(effects
 				(font
@@
 		)
 		(property "Datasheet" ""
-			(at 165.1 88.265 0)
+			(at 156.845 86.995 0)
 			(effects
 				(font
@@
 		)
 		(property "Description" "Power symbol creates a global label with name \"GND\" , ground"
-			(at 165.1 88.265 0)
+			(at 156.845 86.995 0)
 			(effects
 				(font
@@
 	(symbol
 		(lib_id "Device:R_Small")
-		(at 159.385 78.74 90)
+		(at 161.29 78.74 90)
 		(unit 1)
 		(exclude_from_sim no)
@@
 		(dnp no)
 		(property "Reference" "R4"
-			(at 159.385 76.835 90)
+			(at 161.29 76.835 90)
 			(effects
 				(font
@@
 		)
 		(property "Value" "15k"
-			(at 159.385 78.74 90)
+			(at 161.29 78.74 90)
 			(effects
 				(font
@@
 		)
 		(property "Footprint" "Resistor_SMD:R_0603_1608Metric"
-			(at 159.385 78.74 0)
+			(at 161.29 78.74 0)
 			(effects
 				(font
@@
 		)
 		(property "Datasheet" "https://jlcpcb.com/api/file/downloadByFileSystemAccessId/8579706381320323072"
-			(at 159.385 78.74 0)
+			(at 161.29 78.74 0)
 			(effects
 				(font
@@
 		)
 		(property "Description" "-55℃~+155℃ 100mW 15kΩ 75V Thick Film Resistor ±1% ±100ppm/℃ 0603 Chip Resistor - Surface Mount ROHS"
-			(at 159.385 78.74 0)
+			(at 161.29 78.74 0)
 			(effects
 				(font
@@
 		)
 		(property "LCSC" "C22809"
-			(at 159.385 78.74 90)
+			(at 161.29 78.74 90)
 			(effects
 				(font
@@
 		)
 		(property "Link" ""
-			(at 159.385 78.74 90)
-			(effects
-				(font
+			(at 161.29 78.74 90)
+			(effects
+				(font

Commit message: to Kicad 10
Parts:
- added D34: SS84, Diode_SMD:D_SMC, symbol Device:D_Schottky
Connections:
- net +12V: now also D34.1 (K); no longer J1.1 (Pin_1)
- new net: D34.2 (A), J1.1 (Pin_1)
Other:
- moved on the sheet: J1
